File: eagle/gatedriver_trafo_sma_compact.brd (EAGLE design)
At the start: 125.7 x 108.5 mm, 36 parts, among them K1 G5V-2, X4 BU-SMA-V

Commit message: Board, code for dac
Parts:
- moved C2 2.55 mm to (71.4, 35.6)
- moved LV1 0.36 mm to (65.8, 9.14)
Routing:
- net N$22: track 23.0 -> 25.6 mm
- net N$25: track 27.4 -> 26.1 mm
Changed lines of the file:
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@@
 <element name="R4" library="rcl" package="0207/12" value="1M" x="104.14" y="87.884" rot="R90"/>
 <element name="R7" library="rcl" package="0207/12" value="1M" x="104.14" y="64.77" rot="R90"/>
-<element name="C2" library="resistor" package="C050-055X075" value="" x="68.834" y="35.306" rot="R90"/>
+<element name="C2" library="resistor" package="C050-055X075" value="" x="71.374" y="35.56" rot="R90"/>
 <element name="U$2" library="transistor-fet" package="TO92-" value="VN0550" x="90.424" y="47.498" rot="R90"/>
 <element name="U$6" library="transistor-fet" package="TO92-" value="VN0550" x="90.424" y="29.718" rot="R90"/>
@@
 <element name="U$4" library="transistor-fet" package="TO92-" value="VP0550" x="90.424" y="83.566" rot="R270"/>
 <element name="U$5" library="transistor-fet" package="TO92-" value="VP0550" x="90.424" y="63.754" rot="R270"/>
-<element name="LV1" library="testpad" package="P1-20Y" value="TPPAD1-20Y" x="65.532" y="8.89">
-<attribute name="TP_SIGNAL_NAME" value="" x="65.532" y="8.89" size="1.778" layer="27" display="off"/>
+<element name="LV1" library="testpad" package="P1-20Y" value="TPPAD1-20Y" x="65.786" y="9.144">
+<attribute name="TP_SIGNAL_NAME" value="" x="65.786" y="9.144" size="1.778" layer="27" display="off"/>
 </element>
 <element name="HV1" library="testpad" package="P1-20Y" value="TPPAD1-20Y" x="65.532" y="102.362" rot="R180">
@@
 <wire x1="51.054" y1="23.114" x2="51.054" y2="25.146" width="1.6764" layer="16"/>
 <wire x1="51.054" y1="25.146" x2="53.086" y2="27.178" width="1.6764" layer="16"/>
-<wire x1="53.086" y1="27.178" x2="63.246" y2="27.178" width="1.6764" layer="16"/>
-<wire x1="63.246" y1="27.178" x2="68.834" y2="32.766" width="1.6764" layer="16"/>
+<wire x1="53.086" y1="27.178" x2="65.532" y2="27.178" width="1.6764" layer="16"/>
+<wire x1="65.532" y1="27.178" x2="71.374" y2="33.02" width="1.6764" layer="16"/>
 </signal>
 <signal name="N$23">
@@
 <signal name="N$25">
 <contactref element="C2" pad="2"/>
-<wire x1="76.2" y1="47.498" x2="68.834" y2="40.132" width="1.6764" layer="16"/>
-<wire x1="68.834" y1="40.132" x2="68.834" y2="37.846" width="1.6764" layer="16"/>
+<wire x1="76.2" y1="47.498" x2="71.374" y2="42.672" width="1.6764" layer="16"/>
+<wire x1="71.374" y1="42.672" x2="71.374" y2="38.1" width="1.6764" layer="16"/>
 <contactref element="D6" pad="C"/>
 <contactref element="U$2" pad="2"/>
@@
 <contactref element="LV1" pad="TP"/>
 <contactref element="D8" pad="C"/>
-<wire x1="65.532" y1="8.89" x2="80.264" y2="9.144" width="1.6764" layer="16"/>
+<wire x1="65.786" y1="9.144" x2="80.264" y2="9.144" width="1.6764" layer="16"/>
 </signal>
 <signal name="N$20">

Commit message: darlington gate resistor, diode stacking
Parts:
- moved R10 4.32 mm to (99.8, 47.0)
- moved R11 4.32 mm to (99.8, 25.7)
- moved R4 4.32 mm to (99.8, 87.9)
- moved R7 4.32 mm to (99.8, 64.8)
Connections:
- new net N$12: D1.A, D9.C
- new net N$13: D10.A, D4.C
- net N$20: no longer D10.A, D4.C
- net N$21: no longer D1.A, D9.C
Routing:
- net N$21: track 96.5 -> 75.4 mm
- net N$20: track 59.9 -> 39.4 mm
- net GND: track 95.3 -> 115.7 mm, vias 0 -> 2
- net N$12: track 0.00 -> 8.89 mm
- net N$13: track 0.00 -> 8.89 mm
- net N$30: track 89.6 -> 94.9 mm
- removed copper zone on layer 1, net GND
Changed lines of the file:
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@@
 <element name="U$1" library="trafo" package="DIL06" value="DA-2320" x="52.07" y="72.898"/>
 <element name="C5" library="resistor" package="C050-055X075" value="" x="68.326" y="73.914" rot="R90"/>
-<element name="R4" library="rcl" package="0207/12" value="1M" x="104.14" y="87.884" rot="R90"/>
-<element name="R7" library="rcl" package="0207/12" value="1M" x="104.14" y="64.77" rot="R90"/>
+<element name="R4" library="rcl" package="0207/12" value="1M" x="99.822" y="87.884" rot="R90"/>
+<element name="R7" library="rcl" package="0207/12" value="1M" x="99.822" y="64.77" rot="R90"/>
 <element name="C2" library="resistor" package="C050-055X075" value="" x="71.374" y="35.56" rot="R90"/>
 <element name="U$2" library="transistor-fet" package="TO92-" value="VN0550" x="90.424" y="47.498" rot="R90"/>
@@
 <element name="U$7" library="trafo" package="DIL06" value="DA-2320" x="51.054" y="26.924"/>
 <element name="C6" library="resistor" package="C050-055X075" value="" x="66.04" y="19.558"/>
-<element name="R10" library="rcl" package="0207/12" value="1M" x="104.14" y="46.99" rot="R90"/>
-<element name="R11" library="rcl" package="0207/12" value="1M" x="104.14" y="25.654" rot="R90"/>
+<element name="R10" library="rcl" package="0207/12" value="1M" x="99.822" y="46.99" rot="R90"/>
+<element name="R11" library="rcl" package="0207/12" value="1M" x="99.822" y="25.654" rot="R90"/>
 <element name="D1" library="diode" package="C1702-15" value="P6KEXXA" x="112.776" y="86.614" rot="R270"/>
 <element name="D4" library="diode" package="C1702-15" value="P6KEXXA" x="120.396" y="26.924" rot="R270"/>
@@
 <wire x1="25.4" y1="32.004" x2="24.384" y2="33.02" width="1.6764" layer="16"/>
 <wire x1="24.384" y1="33.02" x2="21.082" y2="33.02" width="1.6764" layer="16"/>
-<polygon width="0.4064" layer="1" isolate="1.4224" orphans="yes" thermals="no" rank="6">
-<vertex x="0" y="108.458"/>
-<vertex x="50.292" y="108.712"/>
-<vertex x="50.546" y="0"/>
-<vertex x="0" y="-0.254"/>
-</polygon>
-<wire x1="81.7118" y1="55.5752" x2="68.7832" y2="55.5752" width="3.81" layer="1"/>
-<wire x1="68.7832" y1="55.5752" x2="56.134" y2="42.926" width="3.81" layer="1"/>
-<wire x1="56.134" y1="42.926" x2="49.53" y2="42.926" width="3.81" layer="1"/>
-<wire x1="49.53" y1="42.926" x2="48.514" y2="41.91" width="3.81" layer="1"/>
+<wire x1="81.7118" y1="55.5752" x2="64.2112" y2="55.5752" width="3.81" layer="16"/>
+<wire x1="64.2112" y1="55.5752" x2="46.228" y2="37.592" width="3.81" layer="16"/>
+<wire x1="29.464" y1="65.024" x2="37.592" y2="65.024" width="1.4224" layer="1"/>
+<wire x1="21.844" y1="65.024" x2="13.716" y2="65.024" width="1.4224" layer="1"/>
+<via x="13.716" y="65.024" extent="1-16" drill="0.6" shape="square"/>
+<via x="37.592" y="65.024" extent="1-16" drill="0.6" shape="square"/>
 </signal>
 <signal name="+15V">
@@
 <contactref element="D9" pad="A"/>
 <wire x1="90.424" y1="53.34" x2="90.424" y2="50.038" width="1.6764" layer="16"/>
-<wire x1="104.14" y1="58.42" x2="104.14" y2="56.388" width="1.6764" layer="16"/>
-<wire x1="104.14" y1="56.388" x2="104.14" y2="53.34" width="1.6764" layer="16"/>
+<wire x1="99.822" y1="58.42" x2="99.822" y2="56.388" width="1.6764" layer="16"/>
+<wire x1="99.822" y1="56.388" x2="99.822" y2="53.34" width="1.6764" layer="16"/>
 <wire x1="120.904" y1="63.754" x2="120.904" y2="53.34" width="1.6764" layer="16"/>
 <wire x1="120.904" y1="53.34" x2="119.126" y2="51.1302" width="1.6764" layer="16"/>
 <wire x1="90.424" y1="61.214" x2="90.424" y2="53.34" width="1.6764" layer="16"/>
-<wire x1="90.424" y1="53.34" x2="103.886" y2="53.34" width="1.6764" layer="16"/>
-<wire x1="103.886" y1="53.34" x2="104.14" y2="56.388" width="1.6764" layer="16"/>
-<wire x1="104.14" y1="53.34" x2="112.776" y2="53.34" width="1.6764" layer="16"/>
+<wire x1="90.424" y1="53.34" x2="99.568" y2="53.34" width="1.6764" layer="16"/>
+<wire x1="99.568" y1="53.34" x2="99.822" y2="56.388" width="1.6764" layer="16"/>
+<wire x1="99.822" y1="53.34" x2="112.776" y2="53.34" width="1.6764" layer="16"/>
 <wire x1="112.776" y1="53.34" x2="120.904" y2="53.34" width="1.6764" layer="16"/>
 <wire x1="112.522" y1="49.784" x2="112.522" y2="53.086" width="1.6764" layer="16"/>
@@
 <wire x1="90.424" y1="86.106" x2="90.18610625" y2="93.718565625" width="1.6764" layer="16"/>
 <wire x1="90.18610625" y1="93.718565625" x2="90.17" y2="94.234" width="1.6764" layer="16"/>
-<wire x1="90.17" y1="94.234" x2="104.14" y2="94.234" width="1.6764" layer="16"/>
-<wire x1="104.14" y1="94.234" x2="112.776" y2="94.234" width="1.6764" layer="16"/>
+<wire x1="90.17" y1="94.234" x2="99.822" y2="94.234" width="1.6764" layer="16"/>
+<wire x1="99.822" y1="94.234" x2="107.188" y2="94.234" width="1.6764" layer="16"/>
 <contactref element="D5" pad="C"/>
+<wire x1="107.188" y1="94.234" x2="112.776" y2="94.234" width="1.6764" layer="16"/>
 <wire x1="68.326" y1="93.726" x2="81.534" y2="93.726" width="1.6764" layer="16"/>
 <wire x1="81.534" y1="93.726" x2="90.18610625" y2="93.726" width="1.6764" layer="16"/>
@@
 <wire x1="52.07" y1="76.708" x2="52.07" y2="74.422" width="1.6764" layer="16"/>
 <wire x1="52.07" y1="74.422" x2="52.578" y2="73.914" width="1.6764" layer="16"/>
-<wire x1="104.14" y1="73.914" x2="104.14" y2="71.12" width="1.6764" layer="16"/>
+<wire x1="99.822" y1="73.914" x2="99.822" y2="71.12" width="1.6764" layer="16"/>
 <wire x1="90.424" y1="81.026" x2="90.424" y2="73.914" width="1.6764" layer="16"/>
 <wire x1="90.424" y1="73.914" x2="90.424" y2="66.294" width="1.6764" layer="16"/>
-<wire x1="104.14" y1="81.534" x2="104.14" y2="78.994" width="1.6764" layer="16"/>
-<wire x1="104.14" y1="73.914" x2="90.424" y2="73.914" width="1.6764" layer="16"/>
-<contactref element="D9" pad="C"/>
-<contactref element="D1" pad="A"/>
-<wire x1="112.776" y1="78.994" x2="120.904" y2="78.994" width="1.6764" layer="16"/>
-<wire x1="112.776" y1="78.994" x2="104.14" y2="78.994" width="1.6764" layer="16"/>
-<wire x1="104.14" y1="78.994" x2="104.14" y2="73.914" width="1.6764" layer="16"/>
+<wire x1="99.822" y1="73.914" x2="90.424" y2="73.914" width="1.6764" layer="16"/>
+<wire x1="99.822" y1="81.534" x2="99.822" y2="73.914" width="1.6764" layer="16"/>
 <contactref element="D2" pad="C"/>
 <wire x1="52.578" y1="73.914" x2="81.788" y2="73.914" width="1.6764" layer="16"/>
@@
 <contactref element="R11" pad="2"/>
 <contactref element="R10" pad="1"/>
-<contactref element="D4" pad="C"/>
-<contactref element="D10" pad="A"/>
 <wire x1="81.788" y1="37.338" x2="90.424" y2="37.338" width="1.6764" layer="16"/>
 <wire x1="90.424" y1="37.338" x2="90.424" y2="44.958" width="1.6764" layer="16"/>
 <wire x1="90.424" y1="37.338" x2="90.424" y2="35.56" width="1.6764" layer="16"/>
 <wire x1="90.424" y1="35.56" x2="90.424" y2="32.258" width="1.6764" layer="16"/>
-<wire x1="120.396" y1="34.544" x2="112.522" y2="34.544" width="1.6764" layer="16"/>
-<wire x1="104.14" y1="40.64" x2="104.14" y2="35.56" width="1.6764" layer="16"/>
-<wire x1="104.14" y1="35.56" x2="104.14" y2="34.544" width="1.6764" layer="16"/>
-<wire x1="112.522" y1="34.544" x2="104.14" y2="34.544" width="1.6764" layer="16"/>
-<wire x1="104.14" y1="32.004" x2="104.14" y2="34.544" width="1.6764" layer="16"/>
-<wire x1="104.14" y1="35.56" x2="90.424" y2="35.56" width="1.6764" layer="16"/>
+<wire x1="99.822" y1="40.64" x2="99.822" y2="35.56" width="1.6764" layer="16"/>
+<wire x1="99.822" y1="32.004" x2="99.822" y2="35.56" width="1.6764" layer="16"/>
+<wire x1="99.822" y1="35.56" x2="90.424" y2="35.56" width="1.6764" layer="16"/>
 </signal>
 <signal name="N$30">
@@
 <contactref element="R11" pad="1"/>
 <wire x1="81.788" y1="19.304" x2="90.424" y2="19.304" width="1.6764" layer="16"/>
-<wire x1="90.424" y1="19.304" x2="104.14" y2="19.304" width="1.6764" layer="16"/>
-<wire x1="104.14" y1="19.304" x2="120.396" y2="19.304" width="1.6764" layer="16"/>
+<wire x1="90.424" y1="19.304" x2="99.822" y2="19.304" width="1.6764" layer="16"/>
+<wire x1="99.822" y1="19.304" x2="105.918" y2="19.304" width="1.6764" layer="16"/>
+<wire x1="105.918" y1="19.304" x2="120.396" y2="19.304" width="1.6764" layer="16"/>
 <wire x1="90.424" y1="27.178" x2="90.424" y2="19.304" width="1.6764" layer="16"/>
 <wire x1="90.424" y1="9.144" x2="90.424" y2="19.304" width="1.6764" layer="16"/>
@@
 <via x="64.516" y="30.734" extent="1-16" drill="0.6" shape="square"/>
 <wire x1="64.516" y1="30.734" x2="53.594" y2="30.734" width="1.6764" layer="16"/>
+<wire x1="105.918" y1="24.638" x2="105.918" y2="19.304" width="1.4224" layer="16"/>
+</signal>
+<signal name="N$12">
+<contactref element="D1" pad="A"/>
+<contactref element="D9" pad="C"/>
+<wire x1="112.776" y1="78.994" x2="121.412" y2="78.994" width="1.4224" layer="16"/>
+<wire x1="121.412" y1="78.994" x2="121.412" y2="78.74" width="1.4224" layer="16"/>
+<wire x1="121.412" y1="78.994" x2="120.904" y2="78.994" width="0" layer="19" extent="16-16"/>
+</signal>
+<signal name="N$13">
+<contactref element="D4" pad="C"/>
+<contactref element="D10" pad="A"/>
+<wire x1="120.396" y1="34.544" x2="112.014" y2="34.544" width="1.4224" layer="16"/>
+<wire x1="112.014" y1="34.544" x2="112.014" y2="34.036" width="1.4224" layer="16"/>
+<wire x1="112.014" y1="34.544" x2="112.522" y2="34.544" width="0" layer="19" extent="16-16"/>
 </signal>
 </signals>
