File: eagle/interface_dac_sma.sch (EAGLE design)
At the start: 28 parts, among them X1 BU-SMA-V

Commit message: code
Parts:
- U$2: value MCP4728DIL4 -> MCP4728DIL; device microchip:MCP4728DIL4 -> microchip:MCP4728DIL
Changed lines of the file:
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@@
 <grid distance="0.1" unitdist="inch" unit="inch" style="lines" multiple="1" display="no" altdistance="0.01" altunitdist="inch" altunit="inch"/>
 <layers>
-<layer number="1" name="Top" color="4" fill="1" visible="yes" active="no"/>
-<layer number="2" name="Route2" color="1" fill="3" visible="yes" active="no"/>
-<layer number="3" name="Route3" color="4" fill="3" visible="yes" active="no"/>
-<layer number="4" name="Route4" color="1" fill="4" visible="yes" active="no"/>
-<layer number="5" name="Route5" color="4" fill="4" visible="yes" active="no"/>
-<layer number="6" name="Route6" color="1" fill="8" visible="yes" active="no"/>
-<layer number="7" name="Route7" color="4" fill="8" visible="yes" active="no"/>
-<layer number="8" name="Route8" color="1" fill="2" visible="yes" active="no"/>
-<layer number="9" name="Route9" color="4" fill="2" visible="yes" active="no"/>
-<layer number="10" name="Route10" color="1" fill="7" visible="yes" active="no"/>
-<layer number="11" name="Route11" color="4" fill="7" visible="yes" active="no"/>
-<layer number="12" name="Route12" color="1" fill="5" visible="yes" active="no"/>
-<layer number="13" name="Route13" color="4" fill="5" visible="yes" active="no"/>
-<layer number="14" name="Route14" color="1" fill="6" visible="yes" active="no"/>
-<layer number="15" name="Route15" color="4" fill="6" visible="yes" active="no"/>
-<layer number="16" name="Bottom" color="1" fill="1" visible="yes" active="no"/>
-<layer number="17" name="Pads" color="2" fill="1" visible="yes" active="no"/>
-<layer number="18" name="Vias" color="2" fill="1" visible="yes" active="no"/>
-<layer number="19" name="Unrouted" color="6" fill="1" visible="yes" active="no"/>
-<layer number="20" name="Dimension" color="15" fill="1" visible="yes" active="no"/>
-<layer number="21" name="tPlace" color="7" fill="1" visible="yes" active="no"/>
-<layer number="22" name="bPlace" color="7" fill="1" visible="yes" active="no"/>
-<layer number="23" name="tOrigins" color="15" fill="1" visible="yes" active="no"/>
-<layer number="24" name="bOrigins" color="15" fill="1" visible="yes" active="no"/>
-<layer number="25" name="tNames" color="7" fill="1" visible="yes" active="no"/>
-<layer number="26" name="bNames" color="7" fill="1" visible="yes" active="no"/>
-<layer number="27" name="tValues" color="7" fill="1" visible="yes" active="no"/>
-<layer number="28" name="bValues" color="7" fill="1" visible="yes" active="no"/>
+<layer number="1" name="Top" color="4" fill="1" visible="no" active="no"/>
+<layer number="2" name="Route2" color="1" fill="3" visible="no" active="no"/>
+<layer number="3" name="Route3" color="4" fill="3" visible="no" active="no"/>
+<layer number="4" name="Route4" color="1" fill="4" visible="no" active="no"/>
+<layer number="5" name="Route5" color="4" fill="4" visible="no" active="no"/>
+<layer number="6" name="Route6" color="1" fill="8" visible="no" active="no"/>
+<layer number="7" name="Route7" color="4" fill="8" visible="no" active="no"/>
+<layer number="8" name="Route8" color="1" fill="2" visible="no" active="no"/>
+<layer number="9" name="Route9" color="4" fill="2" visible="no" active="no"/>
+<layer number="10" name="Route10" color="1" fill="7" visible="no" active="no"/>
+<layer number="11" name="Route11" color="4" fill="7" visible="no" active="no"/>
+<layer number="12" name="Route12" color="1" fill="5" visible="no" active="no"/>
+<layer number="13" name="Route13" color="4" fill="5" visible="no" active="no"/>
+<layer number="14" name="Route14" color="1" fill="6" visible="no" active="no"/>
+<layer number="15" name="Route15" color="4" fill="6" visible="no" active="no"/>
+<layer number="16" name="Bottom" color="1" fill="1" visible="no" active="no"/>
+<layer number="17" name="Pads" color="2" fill="1" visible="no" active="no"/>
+<layer number="18" name="Vias" color="2" fill="1" visible="no" active="no"/>
+<layer number="19" name="Unrouted" color="6" fill="1" visible="no" active="no"/>
+<layer number="20" name="Dimension" color="15" fill="1" visible="no" active="no"/>
+<layer number="21" name="tPlace" color="7" fill="1" visible="no" active="no"/>
+<layer number="22" name="bPlace" color="7" fill="1" visible="no" active="no"/>
+<layer number="23" name="tOrigins" color="15" fill="1" visible="no" active="no"/>
+<layer number="24" name="bOrigins" color="15" fill="1" visible="no" active="no"/>
+<layer number="25" name="tNames" color="7" fill="1" visible="no" active="no"/>
+<layer number="26" name="bNames" color="7" fill="1" visible="no" active="no"/>
+<layer number="27" name="tValues" color="7" fill="1" visible="no" active="no"/>
+<layer number="28" name="bValues" color="7" fill="1" visible="no" active="no"/>
 <layer number="29" name="tStop" color="7" fill="3" visible="no" active="no"/>
 <layer number="30" name="bStop" color="7" fill="6" visible="no" active="no"/>
@@
 <layer number="35" name="tGlue" color="7" fill="4" visible="no" active="no"/>
 <layer number="36" name="bGlue" color="7" fill="5" visible="no" active="no"/>
-<layer number="37" name="tTest" color="7" fill="1" visible="yes" active="no"/>
-<layer number="38" name="bTest" color="7" fill="1" visible="yes" active="no"/>
+<layer number="37" name="tTest" color="7" fill="1" visible="no" active="no"/>
+<layer number="38" name="bTest" color="7" fill="1" visible="no" active="no"/>
 <layer number="39" name="tKeepout" color="4" fill="11" visible="no" active="no"/>
 <layer number="40" name="bKeepout" color="1" fill="11" visible="no" active="no"/>
@@
 <layer number="44" name="Drills" color="7" fill="1" visible="no" active="no"/>
 <layer number="45" name="Holes" color="7" fill="1" visible="no" active="no"/>
-<layer number="46" name="Milling" color="3" fill="1" visible="yes" active="no"/>
-<layer number="47" name="Measures" color="7" fill="1" visible="yes" active="no"/>
-<layer number="48" name="Document" color="7" fill="1" visible="yes" active="no"/>
-<layer number="49" name="Reference" color="7" fill="1" visible="yes" active="no"/>
-<layer number="50" name="dxf" color="7" fill="1" visible="yes" active="no"/>
-<layer number="51" name="tDocu" color="7" fill="1" visible="yes" active="no"/>
-<layer number="52" name="bDocu" color="7" fill="1" visible="yes" active="no"/>
-<layer number="53" name="tGND_GNDA" color="7" fill="9" visible="yes" active="no"/>
-<layer number="54" name="bGND_GNDA" color="1" fill="9" visible="yes" active="no"/>
-<layer number="56" name="wert" color="7" fill="1" visible="yes" active="no"/>
+<layer number="46" name="Milling" color="3" fill="1" visible="no" active="no"/>
+<layer number="47" name="Measures" color="7" fill="1" visible="no" active="no"/>
+<layer number="48" name="Document" color="7" fill="1" visible="no" active="no"/>
+<layer number="49" name="Reference" color="7" fill="1" visible="no" active="no"/>
+<layer number="50" name="dxf" color="7" fill="1" visible="no" active="no"/>
+<layer number="51" name="tDocu" color="7" fill="1" visible="no" active="no"/>
+<layer number="52" name="bDocu" color="7" fill="1" visible="no" active="no"/>
+<layer number="53" name="tGND_GNDA" color="7" fill="9" visible="no" active="no"/>
+<layer number="54" name="bGND_GNDA" color="1" fill="9" visible="no" active="no"/>
+<layer number="56" name="wert" color="7" fill="1" visible="no" active="no"/>
 <layer number="90" name="Modules" color="5" fill="1" visible="yes" active="yes"/>
 <layer number="91" name="Nets" color="2" fill="1" visible="yes" active="yes"/>
@@
 <part name="CONTROLHV" library="con-molex" deviceset="KK-156-4" device=""/>
 <part name="GND2" library="supply1" deviceset="GND" device=""/>
-<part name="U$2" library="microchip" deviceset="MCP4728" device="DIL4" value="MCP4728DIL4"/>
+<part name="U$2" library="microchip" deviceset="MCP4728" device="DIL" value="MCP4728DIL"/>
 <part name="P+1" library="supply1" deviceset="VCC" device=""/>
 <part name="GND5" library="supply1" deviceset="GND" device=""/>

Commit message: add iso1540
Parts:
- removed R4, R5: 1k, rcl:R-US_0207/12
- added IC1: ISO1540, texas:ISO1540
- R1, R2: value 100 -> 1.5k; device rcl:R-US_0207/12 -> resistor:R-US_0207/12
Connections:
- removed net N$4: OK1D.C, R1.1
- removed net N$5: OK1C.C, R2.1
- net A+5: now also IC1.VCC1
- net AGND: now also IC1.GND1; no longer R1.2, R2.2
- net GND: now also IC1.GND2; no longer R4.2, R5.2
- net SCL: now also IC1.SCL1; no longer OK1C.A
- net SCL_OUT: now also IC1.SCL2, R2.1; no longer OK1C.EMI, R5.1
- net SDA: now also IC1.SDA1; no longer OK1D.A
- net SDA_OUT: now also IC1.SDA2, R1.1; no longer OK1D.EMI, R4.1
- net VCC: now also IC1.VCC2, R1.2, R2.2; no longer OK1C.COL, OK1D.COL
Other:
- moved on the sheet: R1, R2
Changed lines of the file:
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@@
 <parts>
 <part name="PCB1" library="E14_Arduino_published" deviceset="ARDUINO_MICRO" device=""/>
-<part name="R1" library="rcl" deviceset="R-US_" device="0207/12" value="100"/>
-<part name="R2" library="rcl" deviceset="R-US_" device="0207/12" value="100"/>
 <part name="R3" library="rcl" deviceset="R-US_" device="0207/12" value="100"/>
 <part name="P+5" library="supply1" deviceset="VCC" device=""/>
@@
 <part name="P+1" library="supply1" deviceset="VCC" device=""/>
 <part name="GND5" library="supply1" deviceset="GND" device=""/>
-<part name="P+3" library="supply1" deviceset="VCC" device=""/>
-<part name="R4" library="rcl" deviceset="R-US_" device="0207/12" value="1k"/>
-<part name="GND6" library="supply1" deviceset="GND" device=""/>
-<part name="P+4" library="supply1" deviceset="VCC" device=""/>
-<part name="R5" library="rcl" deviceset="R-US_" device="0207/12" value="1k"/>
-<part name="GND7" library="supply1" deviceset="GND" device=""/>
 <part name="U$4" library="maxim" deviceset="MAX9650" device="DIL" value="MAX9650DIL"/>
 <part name="P+7" library="supply2" deviceset="+12V" device=""/>
@@
 <part name="GND8" library="supply1" deviceset="GND" device=""/>
 <part name="OK1" library="optocoupler" deviceset="PS2501" device="&quot;"/>
+<part name="IC1" library="texas" deviceset="ISO1540" device=""/>
+<part name="GND23" library="supply1" deviceset="GND" device=""/>
+<part name="P+6" library="supply1" deviceset="VCC" device=""/>
+<part name="R1" library="resistor" deviceset="R-US_" device="0207/12" value="1.5k"/>
+<part name="R2" library="resistor" deviceset="R-US_" device="0207/12" value="1.5k"/>
 </parts>
 <sheets>
@@
 <instances>
 <instance part="PCB1" gate="G$1" x="27.94" y="81.28"/>
-<instance part="R1" gate="G$1" x="10.16" y="45.72" rot="R180"/>
-<instance part="R2" gate="G$1" x="10.16" y="2.54" rot="R180"/>
 <instance part="R3" gate="G$1" x="10.16" y="-38.1" rot="R180"/>
 <instance part="P+5" gate="VCC" x="88.9" y="38.1"/>
@@
 <instance part="P+1" gate="VCC" x="104.14" y="106.68"/>
 <instance part="GND5" gate="1" x="139.7" y="106.68" rot="R180"/>
-<instance part="P+3" gate="VCC" x="43.18" y="45.72" rot="R270"/>
-<instance part="R4" gate="G$1" x="45.72" y="40.64"/>
-<instance part="GND6" gate="1" x="53.34" y="40.64" rot="R90"/>
-<instance part="P+4" gate="VCC" x="43.18" y="2.54" rot="R270"/>
-<instance part="R5" gate="G$1" x="45.72" y="-2.54"/>
-<instance part="GND7" gate="1" x="53.34" y="-2.54" rot="R90"/>
 <instance part="U$4" gate="G$2" x="170.18" y="68.58"/>
 <instance part="P+7" gate="+12V" x="167.64" y="78.74"/>
@@
 <instance part="OK1" gate="A" x="27.94" y="-76.2"/>
 <instance part="OK1" gate="B" x="27.94" y="-40.64"/>
-<instance part="OK1" gate="C" x="27.94" y="0"/>
-<instance part="OK1" gate="D" x="27.94" y="43.18"/>
+<instance part="IC1" gate="G$1" x="27.94" y="27.94"/>
+<instance part="GND23" gate="1" x="43.18" y="22.86" rot="R90"/>
+<instance part="P+6" gate="VCC" x="40.64" y="40.64"/>
+<instance part="R1" gate="G$1" x="48.26" y="33.02" rot="R90"/>
+<instance part="R2" gate="G$1" x="55.88" y="30.48" rot="R90"/>
 </instances>
 <busses>
 </busses>
 <nets>
-<net name="N$4" class="0">
-<segment>
-<pinref part="R1" gate="G$1" pin="1"/>
-<wire x1="15.24" y1="45.72" x2="17.78" y2="45.72" width="0.1524" layer="91"/>
-<pinref part="OK1" gate="D" pin="C"/>
-</segment>
-</net>
-<net name="N$5" class="0">
-<segment>
-<pinref part="R2" gate="G$1" pin="1"/>
-<wire x1="17.78" y1="2.54" x2="15.24" y2="2.54" width="0.1524" layer="91"/>
-<pinref part="OK1" gate="C" pin="C"/>
-</segment>
-</net>
 <net name="N$10" class="0">
 <segment>
@@
 </segment>
 <segment>
-<pinref part="R4" gate="G$1" pin="2"/>
-<pinref part="GND6" gate="1" pin="GND"/>
-</segment>
-<segment>
-<pinref part="R5" gate="G$1" pin="2"/>
-<pinref part="GND7" gate="1" pin="GND"/>
-</segment>
-<segment>
 <pinref part="R6" gate="G$1" pin="1"/>
 <pinref part="GND9" gate="1" pin="GND"/>
@@
 <pinref part="GND3" gate="1" pin="GND"/>
 <pinref part="OK1" gate="B" pin="EMI"/>
+</segment>
+<segment>
+<pinref part="IC1" gate="G$1" pin="GND2"/>
+<pinref part="GND23" gate="1" pin="GND"/>
 </segment>
 </net>
@@
 </segment>
 <segment>
-<pinref part="P+3" gate="VCC" pin="VCC"/>
-<wire x1="40.64" y1="45.72" x2="35.56" y2="45.72" width="0.1524" layer="91"/>
-<pinref part="OK1" gate="D" pin="COL"/>
-</segment>
-<segment>
-<pinref part="P+4" gate="VCC" pin="VCC"/>
-<wire x1="40.64" y1="2.54" x2="35.56" y2="2.54" width="0.1524" layer="91"/>
-<pinref part="OK1" gate="C" pin="COL"/>
+<pinref part="IC1" gate="G$1" pin="VCC2"/>
+<pinref part="P+6" gate="VCC" pin="VCC"/>
+<wire x1="40.64" y1="38.1" x2="40.64" y2="30.48" width="0.1524" layer="91"/>
+<pinref part="R1" gate="G$1" pin="2"/>
+<wire x1="40.64" y1="38.1" x2="48.26" y2="38.1" width="0.1524" layer="91"/>
+<wire x1="48.26" y1="38.1" x2="55.88" y2="38.1" width="0.1524" layer="91"/>
+<pinref part="R2" gate="G$1" pin="2"/>
+<wire x1="55.88" y1="38.1" x2="55.88" y2="35.56" width="0.1524" layer="91"/>
 </segment>
 </net>
@@
 <net name="AGND" class="0">
 <segment>
-<pinref part="R1" gate="G$1" pin="2"/>
-<pinref part="R2" gate="G$1" pin="2"/>
-<wire x1="5.08" y1="45.72" x2="5.08" y2="2.54" width="0.1524" layer="91"/>
 <pinref part="R3" gate="G$1" pin="2"/>
-<wire x1="5.08" y1="25.4" x2="5.08" y2="2.54" width="0.1524" layer="91"/>
-<wire x1="5.08" y1="2.54" x2="5.08" y2="-38.1" width="0.1524" layer="91"/>
 <wire x1="5.08" y1="-38.1" x2="5.08" y2="-73.66" width="0.1524" layer="91"/>
 <pinref part="R18" gate="G$1" pin="2"/>
@@
 <segment>
 <pinref part="PCB1" gate="G$1" pin="GND."/>
-<wire x1="43.18" y1="63.5" x2="43.18" y2="55.88" width="0.1524" layer="91"/>
+<wire x1="43.18" y1="63.5" x2="43.18" y2="53.34" width="0.1524" layer="91"/>
+</segment>
+<segment>
+<wire x1="10.16" y1="22.86" x2="15.24" y2="22.86" width="0.1524" layer="91"/>
+<pinref part="IC1" gate="G$1" pin="GND1"/>
 </segment>
 </net>
@@
 <wire x1="38.1" y1="63.5" x2="38.1" y2="55.88" width="0.1524" layer="91"/>
 </segment>
+<segment>
+<wire x1="10.16" y1="30.48" x2="15.24" y2="30.48" width="0.1524" layer="91"/>
+<pinref part="IC1" gate="G$1" pin="VCC1"/>
+</segment>
 </net>
 <net name="D10" class="0">
@@
 </segment>
 <segment>
-<wire x1="17.78" y1="40.64" x2="12.7" y2="40.64" width="0.1524" layer="91"/>
-<pinref part="OK1" gate="D" pin="A"/>
+<wire x1="15.24" y1="27.94" x2="10.16" y2="27.94" width="0.1524" layer="91"/>
+<pinref part="IC1" gate="G$1" pin="SDA1"/>
 </segment>
 </net>
@@
 </segment>
 <segment>
-<wire x1="17.78" y1="-2.54" x2="12.7" y2="-2.54" width="0.1524" layer="91"/>
-<pinref part="OK1" gate="C" pin="A"/>
+<wire x1="15.24" y1="25.4" x2="10.16" y2="25.4" width="0.1524" layer="91"/>
+<pinref part="IC1" gate="G$1" pin="SCL1"/>
 </segment>
 </net>
 <net name="SDA_OUT" class="0">
-<segment>
-<pinref part="R4" gate="G$1" pin="1"/>
-<wire x1="40.64" y1="40.64" x2="35.56" y2="40.64" width="0.1524" layer="91"/>
-<pinref part="OK1" gate="D" pin="EMI"/>
-</segment>
 <segment>
 <wire x1="104.14" y1="83.82" x2="99.06" y2="83.82" width="0.1524" layer="91"/>
 <pinref part="U$2" gate="G$1" pin="SDA"/>
 </segment>
+<segment>
+<wire x1="48.26" y1="27.94" x2="40.64" y2="27.94" width="0.1524" layer="91"/>
+<pinref part="IC1" gate="G$1" pin="SDA2"/>
+<pinref part="R1" gate="G$1" pin="1"/>
+</segment>
 </net>
 <net name="SCL_OUT" class="0">
-<segment>
-<pinref part="R5" gate="G$1" pin="1"/>
-<wire x1="40.64" y1="-2.54" x2="35.56" y2="-2.54" width="0.1524" layer="91"/>
-<pinref part="OK1" gate="C" pin="EMI"/>
-</segment>
 <segment>
 <wire x1="104.14" y1="93.98" x2="99.06" y2="93.98" width="0.1524" layer="91"/>
 <pinref part="U$2" gate="G$1" pin="SCL"/>
 </segment>
-</net>
+<segment>
+<pinref part="IC1" gate="G$1" pin="SCL2"/>
+<pinref part="R2" gate="G$1" pin="1"/>
+<wire x1="40.64" y1="25.4" x2="55.88" y2="25.4" width="0.1524" layer="91"/>
+</segment>
+</net>

Commit message: Code debug, add darlingtons to HV input
Parts:
- added T1, T2, T3: TIP122V, transistor-npn:TIP122V
Connections:
- new net N$4: CONTROLHV-1.S, R8.1, T1.E
- new net N$5: T1.B, U$4.OUT
- new net N$6: CONTROLHV-2.S, R10.1, T2.E
- net +12V: now also T1.C, T2.C, T3.C
- net N$11: now also CONTROLHV-3.S, R12.1, T3.E; no longer CONTROLHV-2.S, R10.1, U$5.OUT
- net N$15: now also T3.B; no longer CONTROLHV-3.S, R12.1
- net N$3: now also T2.B, U$5.OUT; no longer CONTROLHV-1.S, R8.1, U$4.OUT
Other:
- moved on the sheet: CONTROLHV-1, CONTROLHV-2, CONTROLHV-3

Commit message: darlington gate resistor, diode stacking
Parts:
- added R14, R4, R5: 14k, resistor:R-US_0207/12
Connections:
- new net N$19: R4.2, U$4.OUT
- new net N$20: R5.2, U$5.OUT
- new net N$21: R14.2, U$6.OUT
- net N$15: now also R14.1; no longer U$6.OUT
- net N$3: now also R4.1, T1.B; no longer T2.B, U$5.OUT
- net N$5: now also R5.1, T2.B; no longer T1.B, U$4.OUT
Other:
- moved on the sheet: CONTROLHV-1, CONTROLHV-2, CONTROLHV-3, T1, T2, T3
