File: eagle/interface_dac_sma_feedback.brd (EAGLE design)
At the start: 119.6 x 108.5 mm, 37 parts, among them K1 G5V-2, X4 BU-SMA-V

Commit message: feedback on hv rails
Parts:
- removed C1, C2, C3, C5, C6: (no value), resistor:C050-055X075
- removed C7: (no value), rcl:C050-030X075
- removed D1, D10, D4, D9: P6KEXXA, diode:C1702-15
- removed D11: 1N4148DO35-10, diode:DO35-10
- removed D14, D2, D5, D6: 4742, diode:ZDIO-10
- removed D7, D8: 1N4004, diode:DO41-10
- removed GND, HV1, LV1, OUT: TPPAD1-20Y, testpad:P1-20Y
- removed K1: G5V-2, relay:G5V-2
- removed POWERGD: (no value), con-molex:KK-156-2
- removed R10, R11: 1M, rcl:0207/12
- removed U$3: UCC27425, texas:DIL08
- removed U$7: DA-2320, trafo:DIL06
- removed X4: BU-SMA-V, con-coax:BU-SMA-V
- added CONTROLGD2: (no value), con-molex:KK-156-2
- added CONTROLHV, CONTROLHVFDBK: (no value), con-molex:KK-156-4
- added IC1: ISO1540, texas:DIL08
- added OK1: PS2501", optocoupler:DIL16
- added PCB1: ARDUINO_MICRO, E14_Arduino_published:ARDUINO_MICRO
- added POWERINTERFACE: (no value), con-molex:KK-156-3
- added R1, R2: 1.5k, resistor:0207/12
- added R14, R5: 14k, resistor:0207/12
- added R16: (no value), pot:SP19L
- added R18, R3: 100, rcl:0207/12
- added R6: 10k, resistor:0207/12
- added T1, T2, T3: TIP122V, transistor-npn:TO220V
- added X1: BU-SMA-V, con-coax:BU-SMA-V
- C4: device resistor:C050-055X075 -> resistor:C075-063X106
- R4: value 1M -> 14k; device rcl:0207/12 -> resistor:0207/12
- R7: value 1M -> 40k; device rcl:0207/12 -> resistor:0207/12
- U$1: value DA-2320 -> LTC6992; device trafo:DIL06 -> linear-technology:DIL06
- U$2: value VN0550 -> MCP4728DIL; device transistor-fet:TO92- -> microchip:DIL10
- U$4, U$5: value VP0550 -> MAX9650DIL; device transistor-fet:TO92- -> maxim:DIL06-4
- U$6: value VN0550 -> MAX9650DIL; device transistor-fet:TO92- -> maxim:DIL06-4
- moved R4 94.9 mm to (5.59, 99.3), turned to 270 degrees
- moved U$4 73.7 mm to (17.4, 93.7)
- moved C4 71.4 mm to (98.3, 62.4)
- moved U$6 65.1 mm to (83.1, 94.4), turned to 270 degrees
- moved U$2 56.1 mm to (42.4, 76.5), turned to 0 degrees
- moved U$5 50.7 mm to (49.7, 93.9)
- moved U$1 36.1 mm to (88.1, 73.2), turned to 270 degrees
- moved R7 33.1 mm to (68.2, 74.4), turned to 0 degrees
- moved CONTROLGD1 29.8 mm to (20.6, 74.7), turned to 180 degrees
Connections:
- removed net +15V: C7.1, D11.C, K1.1, K1.8, K1.9, POWERGD.1, U$3.6
- removed net ENSW: CONTROLGD1.1, D11.A, K1.16
- removed net N$22: C2.1, U$7.2
- removed net N$23: C6.1, U$7.3
- removed net N$25: C2.2, D6.C, U$2.2
- removed net N$27: C6.2, D14.C, U$6.2
- removed net N$29: D7.A, HV1.TP
- removed net N$30: D14.A, D4.A, D8.A, R11.1, U$6.3, U$7.4
- new net +12V: POWERINTERFACE.1, T1.2, T2.2, T3.2, U$4.6, U$5.6, U$6.6
- new net A+5: IC1.1, PCB1.+5V
- new net AGND: IC1.4, PCB1.GND., R18.2, R3.2
- new net D10: PCB1.D10
- new net D11: PCB1.D11
- new net D4: PCB1.D4
- new net D7: PCB1.D7
- new net D8: PCB1.D8
- new net ENSW1: CONTROLGD1.1, OK1.14
- new net ENSW2: CONTROLGD2.1, OK1.16
- new net N$12: R16.E, U$1.SET
- new net N$19: R4.2, U$4.1
- new net N$20: R5.2, U$5.1
- new net N$8: CONTROLHVFDBK.1, U$4.4
- new net PWM5: PCB1.D5
- new net PWM6: OK1.3, PCB1.D6
- new net PWM9: OK1.1, PCB1.D9
- new net SCL: IC1.3, PCB1.D3
- new net SCL_OUT: IC1.6, R2.1, U$2.2
- new net SDA: IC1.2, PCB1.D2
- new net SDA_OUT: IC1.7, R1.1, U$2.3
- new net VCC: C4.1, IC1.8, POWERINTERFACE.2, R1.2, R2.2, U$1.VCC, U$2.1
- net GND: now also C4.2, CONTROLGD2.2, CONTROLHV.4, CONTROLHVFDBK.4, IC1.5, OK1.13, OK1.15, POWERINTERFACE.3, R16.A, R16.S, R6.1, U$1.DIV, U$1.GND, U$2.10, U$2.4, U$4.2, U$5.2, U$6.2, X1.2, X1.3, X1.4, X1.5; no longer C7.2, GND.TP, K1.11, K1.6, POWERGD.2, U$1.6, U$3.3, U$7.6, X4.2, X4.3, X4.4, X4.5
- net N$1: now also R7.1, U$2.6; no longer U$3.2, U$3.4, X4.1
- net N$10: now also OK1.4, R3.1; no longer D8.C, LV1.TP
- net N$11: now also CONTROLHV.3, T3.3; no longer C1.2, D2.A, U$5.2
- net N$13: now also U$1.OUT, X1.1; no longer D10.A, D4.C, D6.A, R10.1, R11.2, U$2.3, U$6.1
- net N$14: now also CONTROLHVFDBK.3, U$6.4; no longer K1.4, U$3.1
- net N$15: now also R14.1, T3.1; no longer K1.13, U$3.8
- net N$16: now also U$2.9, U$4.3; no longer C5.2, D5.A, U$4.2
- net N$17: now also U$2.8, U$5.3; no longer D1.C, D5.C, D7.C, R4.2, U$1.4, U$4.3
- net N$18: now also U$2.7, U$6.3; no longer D1.A, D2.C, D9.C, R4.1, R7.2, U$1.5, U$4.1, U$5.3
- net N$2: now also R6.2, R7.2, U$1.MOD; no longer C3.1, U$3.7
- net N$21: now also R14.2, U$6.1; no longer D10.C, D9.A, OUT.TP, R10.2, R7.1, U$2.1, U$5.1
- net N$3: now also R4.1, T1.1; no longer C3.2, U$1.1
- net N$4: now also CONTROLHV.1, T1.3; no longer C4.1, U$3.5
- net N$5: now also R5.1, T2.1; no longer C1.1, U$1.2
- net N$6: now also CONTROLHV.2, T2.3; no longer C4.2, U$7.1
- net N$7: now also OK1.2, R18.1; no longer C5.1, U$1.3
- net N$9: now also CONTROLHVFDBK.2, U$5.4; no longer U$7.5
Routing:
- net VCC: track 0.00 -> 175.2 mm, vias 0 -> 2
- net +12V: track 0.00 -> 171.2 mm
- net N$30: track 83.5 -> 0.00 mm, vias 2 -> 0
- net +15V: track 77.9 -> 0.00 mm
- net N$17: track 85.6 -> 13.3 mm
- net N$8: track 0.00 -> 68.5 mm, vias 0 -> 2
- net GND: track 115.7 -> 48.1 mm, vias 2 -> 0
- net AGND: track 0.00 -> 63.8 mm
- net A+5: track 0.00 -> 51.8 mm
- net N$11: track 21.8 -> 73.5 mm
- net N$18: track 90.7 -> 40.6 mm
- net N$13: track 55.6 -> 8.72 mm
- net SCL_OUT: track 0.00 -> 46.8 mm, vias 0 -> 2
- net N$21: track 54.6 -> 10.8 mm
- net N$6: track 7.37 -> 46.1 mm
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- added copper zone on layer 16, net AGND
Other:
- board size 119.6 x 108.5 mm -> 109.5 x 142.9 mm
