File: eagle/hvreg_feedback_3PS.brd (EAGLE design)
At the start: 152.4 x 101.6 mm, 20 parts

Commit message: use SW on one side, DC on the other. HV feedback. Positive only
Parts:
- removed CONTROLHV, FDBKHV: (no value), con-molex:KK-156-3
- added C10: (no value), rcl:C050-030X075
- added C8: .01u, rcl:C075-042X103
- added C9: 1u, rcl:C225-108X268
- added D3, D4: 1n4733, diode:ZDIO-10
- added LV+, LV-: TPPAD1-20Y, testpad:P1-20Y
- added R4, R6: 2M, resistor:0207/12
- added R5, R8: (no value), pot:SP19L
- added U$3: EMCO-F104PIN, dc-dc-converter:EMCO-F
- C5, C6: device rcl:C275-113X316 -> rcl:C225-108X268
- moved C4 196.4 mm to (5.08, -118.4), turned to 0 degrees
- moved C7 193.4 mm to (13.5, -98.6), turned to 0 degrees
- moved HV- 165.4 mm to (16.0, -62.0)
Connections:
- new net N$10: C10.1, U$3.P$1
- new net N$11: D4.A, R6.2, R8.A
- new net N$7: C8.1, C9.1, HV-.TP, R4.1
- new net N$9: D3.A, R4.2, R5.A
- net GND: now also C10.2, C8.2, C9.2, D3.C, D4.C, R5.E, R5.S, R8.E, R8.S, U$3.P$2, U$3.P$3; no longer CONTROLHV.2, FDBKHV.2
- net N$2: now also LV+.TP
- net N$3: no longer FDBKHV.1
- net N$4: no longer CONTROLHV.1
- net N$5: no longer CONTROLHV.3
- net N$6: now also LV-.TP, R6.1; no longer HV-.TP, U$2.P$4
- net N$8: no longer FDBKHV.3
Routing:
- net GND: track 349.9 -> 270.9 mm
- net N$6: track 72.7 -> 0.00 mm
- net N$3: track 103.6 -> 60.3 mm
- net N$4: track 55.3 -> 50.9 mm
- net N$2: track 62.3 -> 60.1 mm
