File: eagle/hvreg_feedback_3PS.sch (EAGLE design)
At the start: 20 parts

Commit message: use SW on one side, DC on the other. HV feedback. Positive only
Parts:
- removed CONTROLHV, FDBKHV: (no value), con-molex:KK-156-3
- added C10: (no value), rcl:C-US050-030X075
- added C8: .01u, rcl:C-US075-042X103
- added C9: 1u, rcl:C-US225-108X268
- added D3, D4: 1n4733, diode:ZENER-DIODEZD-10
- added LV+, LV-: TPPAD1-20Y, testpad:TPPAD1-20Y
- added R4, R6: 2M, resistor:R-US_0207/12
- added R5, R8: (no value), pot:TRIM_US-B90P
- added U$3: EMCO-F104PIN, dc-dc-converter:EMCO-F104PIN
- C5, C6: device rcl:C-US275-113X316 -> rcl:C-US225-108X268
Connections:
- new net N$10: C10.1, U$3.+VIN
- new net N$11: D4.A, R6.2, R8.A
- new net N$7: C8.1, C9.1, HV-.TP, R4.1
- new net N$9: D3.A, R4.2, R5.A
- net GND: now also C10.2, C8.2, C9.2, D3.C, D4.C, R5.E, R5.S, R8.E, R8.S, U$3.+VOUT, U$3.-VIN; no longer CONTROLHV-2.S, FDBKHV-2.S
- net N$2: now also LV+.TP
- net N$3: no longer FDBKHV-1.S
- net N$4: no longer CONTROLHV-1.S
- net N$5: no longer CONTROLHV-3.S
- net N$6: now also LV-.TP, R6.1; no longer HV-.TP, U$2.-VOUT
- net N$8: no longer FDBKHV-3.S
Other:
- moved on the sheet: C12, C4, C6, C7, D2, HV-, R3, R7
