File: eagle/ifacegdcombo.brd (EAGLE design)
At the start: 192.8 x 133.3 mm, 71 parts, among them IC1 ISO1540, K1 G5V-2, T1 TIP122V, T3 TIP122V, X1 BU-SMA-V, X4 BU-SMA-V

Commit message: 4pcb upload
Parts:
- added D12, D3, D7, D8: 1N4148DO35-10, diode:DO35-10
- moved R6 2.30 mm to (61.5, 57.9)
- moved R8 1.52 mm to (61.5, 78.5)
- moved R9 1.52 mm to (61.0, 53.1)
- moved R12 1.02 mm to (61.2, 33.8)
- moved R1 0.25 mm to (66.5, 69.1)
Connections:
- net N$10: now also D3.A
- net N$11: now also D12.A
- net N$12: now also D7.C
- net N$16: now also D7.A
- net N$25: now also D8.C
- net N$251: now also D8.A
- net N$27: now also D12.C
- net N$8: now also D3.C
Routing:
- net N$8: track 13.7 -> 15.7 mm
- net N$10: track 12.0 -> 13.6 mm
- net N$25: track 14.9 -> 16.5 mm
- net N$251: track 8.89 -> 10.4 mm
- net N$16: track 13.6 -> 15.1 mm
- net N$12: track 14.0 -> 15.5 mm
- net N$27: track 15.2 -> 16.2 mm
- net N$11: track 8.89 -> 9.91 mm
Changed lines of the file:
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@@
 <element name="D14" library="diode" package="ZDIO-10" value="4742" x="56.134" y="23.622" rot="R270"/>
 <element name="C7" library="rcl" package="C050-030X075" value="" x="6.858" y="83.312" rot="R270"/>
-<element name="R1" library="rcl" package="0207/10" value="50k" x="66.294" y="69.088" rot="R90"/>
+<element name="R1" library="rcl" package="0207/10" value="50k" x="66.548" y="69.088" rot="R90"/>
 <element name="R2" library="rcl" package="0207/10" value="50k" x="66.548" y="89.408" rot="R90"/>
 <element name="R3" library="rcl" package="0207/10" value="50k" x="66.04" y="42.672" rot="R270"/>
 <element name="R5" library="rcl" package="0207/10" value="50k" x="66.294" y="23.622" rot="R270"/>
-<element name="R6" library="rcl" package="0207/10" value="70" x="61.214" y="60.198"/>
-<element name="R8" library="rcl" package="0207/10" value="70" x="61.468" y="80.01"/>
-<element name="R9" library="rcl" package="0207/10" value="70" x="60.96" y="51.562"/>
-<element name="R12" library="rcl" package="0207/10" value="70" x="61.214" y="32.766"/>
+<element name="R6" library="rcl" package="0207/10" value="70" x="61.468" y="57.912"/>
+<element name="R8" library="rcl" package="0207/10" value="70" x="61.468" y="78.486"/>
+<element name="R9" library="rcl" package="0207/10" value="70" x="60.96" y="53.086"/>
+<element name="R12" library="rcl" package="0207/10" value="70" x="61.214" y="33.782"/>
 <element name="R13" library="rcl" package="0207/10" value="70" x="35.052" y="60.198" rot="R270"/>
 <element name="R14" library="rcl" package="0207/10" value="1M" x="26.924" y="14.478" rot="R180"/>
@@
 </element>
 <element name="C9" library="resistor" package="C102-064X133" value="10p" x="55.626" y="7.874" rot="R180"/>
+<element name="D3" library="diode" package="DO35-10" value="1N4148DO35-10" x="61.468" y="61.214" rot="R180"/>
+<element name="D7" library="diode" package="DO35-10" value="1N4148DO35-10" x="61.468" y="81.534" rot="R180"/>
+<element name="D8" library="diode" package="DO35-10" value="1N4148DO35-10" x="60.96" y="50.038"/>
+<element name="D12" library="diode" package="DO35-10" value="1N4148DO35-10" x="61.214" y="30.988"/>
 <element name="PCB1" library="E14_Arduino_published" package="ARDUINO_MICRO" value="ARDUINO_MICRO" x="114.681" y="5.969"/>
 <element name="POWERINTERFACE" library="con-molex" package="KK-156-3" value="" x="172.1104" y="117.1448">
@@
 <contactref element="R9" pad="1"/>
 <wire x1="48.006" y1="38.862" x2="55.88" y2="46.736" width="1.6764" layer="16"/>
-<wire x1="55.88" y1="47.752" x2="55.88" y2="51.562" width="1.6764" layer="16"/>
+<wire x1="55.88" y1="47.752" x2="55.88" y2="53.086" width="1.6764" layer="16"/>
+<contactref element="D8" pad="C"/>
+<wire x1="55.88" y1="47.752" x2="55.88" y2="50.038" width="0" layer="19" extent="1-1"/>
 <wire x1="55.88" y1="46.736" x2="55.88" y2="47.752" width="0" layer="19" extent="16-16"/>
 </signal>
@@
 <contactref element="D14" pad="C"/>
 <wire x1="50.038" y1="20.066" x2="56.134" y2="26.162" width="1.6764" layer="16"/>
-<wire x1="56.134" y1="26.162" x2="56.134" y2="32.766" width="1.6764" layer="16"/>
+<wire x1="56.134" y1="26.162" x2="56.134" y2="33.782" width="1.6764" layer="16"/>
+<contactref element="D12" pad="C"/>
+<wire x1="56.134" y1="28.702" x2="56.134" y2="30.988" width="0" layer="19" extent="1-1"/>
 <wire x1="56.134" y1="26.162" x2="56.134" y2="28.702" width="0" layer="19" extent="16-16"/>
 </signal>
@@
 <wire x1="54.61" y1="81.788" x2="56.134" y2="81.788" width="1.6764" layer="16"/>
 <wire x1="56.134" y1="81.788" x2="56.388" y2="81.534" width="1.6764" layer="16"/>
-<wire x1="56.388" y1="81.534" x2="56.388" y2="80.01" width="1.6764" layer="16"/>
+<wire x1="56.388" y1="81.534" x2="56.388" y2="78.486" width="1.6764" layer="16"/>
 <wire x1="56.388" y1="84.328" x2="56.388" y2="81.534" width="1.6764" layer="16"/>
+<contactref element="D7" pad="A"/>
 </signal>
 <signal name="N$17">
@@
 <wire x1="37.592" y1="76.962" x2="37.592" y2="74.676" width="1.4224" layer="16"/>
 <wire x1="37.592" y1="74.676" x2="38.862" y2="74.168" width="1.4224" layer="16"/>
-<wire x1="38.862" y1="74.168" x2="66.294" y2="74.168" width="1.4224" layer="16"/>
+<wire x1="38.862" y1="74.168" x2="66.548" y2="74.168" width="1.4224" layer="16"/>
 <wire x1="73.66" y1="81.788" x2="73.66" y2="74.168" width="1.6764" layer="16"/>
 <wire x1="73.66" y1="74.168" x2="73.66" y2="66.548" width="1.6764" layer="16"/>
@@
 <contactref element="R1" pad="2"/>
 <wire x1="56.388" y1="74.422" x2="56.642" y2="74.168" width="1.6764" layer="16"/>
-<wire x1="56.642" y1="74.168" x2="66.294" y2="74.168" width="1.6764" layer="16"/>
-<wire x1="66.294" y1="74.168" x2="73.66" y2="74.168" width="1.6764" layer="16"/>
+<wire x1="56.642" y1="74.168" x2="66.548" y2="74.168" width="1.6764" layer="16"/>
+<wire x1="66.548" y1="74.168" x2="73.66" y2="74.168" width="1.6764" layer="16"/>
 </signal>
 <signal name="N$8">
@@
 <contactref element="R1" pad="1"/>
 <contactref element="R6" pad="2"/>
-<wire x1="66.294" y1="60.198" x2="66.294" y2="64.008" width="1.6764" layer="16"/>
-<wire x1="76.2" y1="64.008" x2="66.294" y2="64.008" width="1.4224" layer="1"/>
+<wire x1="66.548" y1="57.912" x2="66.548" y2="64.008" width="1.6764" layer="16"/>
+<wire x1="76.2" y1="64.008" x2="66.548" y2="64.008" width="1.4224" layer="1"/>
+<contactref element="D3" pad="C"/>
+<wire x1="66.548" y1="64.008" x2="66.548" y2="61.214" width="0" layer="19" extent="1-1"/>
 </signal>
 <signal name="N$10">
@@
 <wire x1="52.07" y1="62.23" x2="56.134" y2="62.23" width="1.6764" layer="16"/>
 <wire x1="56.134" y1="62.23" x2="56.388" y2="62.484" width="1.6764" layer="16"/>
-<wire x1="56.388" y1="62.484" x2="56.388" y2="62.738" width="1.6764" layer="16"/>
-<wire x1="56.388" y1="62.738" x2="56.388" y2="64.262" width="1.6764" layer="16"/>
-<wire x1="56.134" y1="60.198" x2="56.388" y2="59.944" width="1.6764" layer="16"/>
-<wire x1="56.388" y1="59.944" x2="56.388" y2="62.484" width="1.6764" layer="16"/>
+<wire x1="56.388" y1="62.484" x2="56.388" y2="64.262" width="1.6764" layer="16"/>
+<wire x1="56.388" y1="57.912" x2="56.388" y2="62.484" width="1.6764" layer="16"/>
+<contactref element="D3" pad="A"/>
+<wire x1="56.134" y1="62.23" x2="56.388" y2="61.214" width="0" layer="19" extent="16-16"/>
 </signal>
 <signal name="N$11">
@@
 <contactref element="U$6" pad="2"/>
 <contactref element="R12" pad="2"/>
-<wire x1="66.294" y1="32.766" x2="66.294" y2="28.702" width="1.6764" layer="16"/>
+<wire x1="66.294" y1="33.782" x2="66.294" y2="28.702" width="1.6764" layer="16"/>
 <wire x1="66.294" y1="28.702" x2="71.12" y2="28.702" width="1.6764" layer="16"/>
+<contactref element="D12" pad="A"/>
+<wire x1="66.294" y1="28.702" x2="66.294" y2="30.988" width="0" layer="19" extent="1-1"/>
 </signal>
 <signal name="N$12">
@@
 <contactref element="R2" pad="1"/>
 <contactref element="R8" pad="2"/>
-<wire x1="66.548" y1="80.01" x2="66.548" y2="84.328" width="1.6764" layer="16"/>
+<wire x1="66.548" y1="78.486" x2="66.548" y2="84.328" width="1.6764" layer="16"/>
 <wire x1="76.2" y1="84.328" x2="66.548" y2="84.328" width="1.4224" layer="1"/>
+<contactref element="D7" pad="C"/>
+<wire x1="66.548" y1="84.328" x2="66.548" y2="81.534" width="0" layer="19" extent="1-1"/>
 </signal>
 <signal name="N$3">
@@
 <contactref element="R9" pad="2"/>
 <contactref element="U$2" pad="2"/>
-<wire x1="66.04" y1="51.562" x2="66.04" y2="47.752" width="1.6764" layer="16"/>
+<wire x1="66.04" y1="53.086" x2="66.04" y2="47.752" width="1.6764" layer="16"/>
 <wire x1="66.04" y1="47.752" x2="71.12" y2="47.752" width="1.6764" layer="16"/>
+<contactref element="D8" pad="A"/>
+<wire x1="66.04" y1="47.752" x2="66.04" y2="50.038" width="0" layer="19" extent="1-1"/>
 </signal>
 <signal name="N$24">
@@
 <polygon width="0.4064" layer="16" spacing="1.4224" isolate="1.4224">
 <vertex x="102.743" y="0.127"/>
-<vertex x="197.104" y="0.127"/>
-<vertex x="197.231" y="46.101"/>
+<vertex x="192.024" y="0.127"/>
+<vertex x="192.151" y="46.101"/>
 <vertex x="102.997" y="45.974"/>
 </polygon>
