File: eagle/interface_dac_sma_feedback_2PS.sch (EAGLE design)
At the start: 25 parts, among them IC1 ISO1540, T1 TIP122V, T3 TIP122V, X1 BU-SMA-V

Commit message: layout fixes
Connections:
- removed net N$7: OK2.A, R18.1
- new net N$6: OK2.C, R18.1
- net PWM9: now also OK2.A; no longer OK2.C
Other:
- moved on the sheet: R18
Changed lines of the file:
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@@
 <instance part="X1" gate="G$1" x="289.56" y="91.44" rot="R90"/>
 <instance part="GND17" gate="1" x="292.1" y="96.52" rot="R180"/>
-<instance part="R18" gate="G$1" x="10.16" y="-73.66" rot="R180"/>
+<instance part="R18" gate="G$1" x="12.7" y="-78.74" rot="R180"/>
 <instance part="GND1" gate="1" x="35.56" y="-81.28"/>
 <instance part="CONTROLGD2" gate="-1" x="53.34" y="-73.66"/>
@@
 <net name="AGND" class="0">
 <segment>
-<wire x1="0" y1="-73.66" x2="5.08" y2="-73.66" width="0.1524" layer="91"/>
+<wire x1="2.54" y1="-78.74" x2="7.62" y2="-78.74" width="0.1524" layer="91"/>
 <pinref part="R18" gate="G$1" pin="2"/>
 </segment>
@@
 </segment>
 <segment>
-<wire x1="17.78" y1="-78.74" x2="12.7" y2="-78.74" width="0.1524" layer="91"/>
-<pinref part="OK2" gate="G$1" pin="C"/>
+<wire x1="17.78" y1="-73.66" x2="12.7" y2="-73.66" width="0.1524" layer="91"/>
+<pinref part="OK2" gate="G$1" pin="A"/>
 </segment>
 </net>
@@
 <pinref part="X1" gate="G$1" pin="1"/>
 <wire x1="289.56" y1="93.98" x2="279.4" y2="93.98" width="0.1524" layer="91"/>
-</segment>
-</net>
-<net name="N$7" class="0">
-<segment>
-<pinref part="R18" gate="G$1" pin="1"/>
-<wire x1="17.78" y1="-73.66" x2="15.24" y2="-73.66" width="0.1524" layer="91"/>
-<pinref part="OK2" gate="G$1" pin="A"/>
 </segment>
 </net>
@@
 </segment>
 </net>
+<net name="N$6" class="0">
+<segment>
+<pinref part="OK2" gate="G$1" pin="C"/>
+<pinref part="R18" gate="G$1" pin="1"/>
+</segment>
+</net>
