File: eagle/gatedriver_trafo_sma_compact_ACDC_ultra.brd (EAGLE design)
At the start: 158.8 x 171.4 mm, 38 parts

Commit message: use lm317, appropriate opamp resistor selection, ultra gatedriver stacks 4 fets
Parts:
- removed C13: .01u, rcl:C102-043X133
- removed C17, C18, C19: .1u, rcl:C102-043X133
- removed CONTROLHV, FDBKHV: (no value), con-molex:KK-156-4
- removed HV+, HV-, LV+, LV-: TPPAD1-20Y, testpad:P1-20Y
- added CONTROLGD1, POWERGD: (no value), con-molex:KK-156-2
- added D10, D13, D15, D20, D21, D9: P6KEXXA, diode:C1702-15
- added D11, D12, D18, D19, D24, D25, D7, D8: 1N4148DO35-10, diode:DO35-10
- added D14, D16, D17, D22, D23, D5, D6: 4742, diode:ZDIO-10
- added HV1, HV2, OUT: TPPAD1-20Y, testpad:P1-20Y
- added K1: G5V-2, relay:G5V-2
- added R10, R11, R14, R15, R16, R22, R23, R28: 1M, rcl:0207/10
- added R12, R13, R19, R20, R21, R26, R27, R6, R8, R9: 70, rcl:0207/10
- added R17, R18, R24, R25: 50k, rcl:0207/10
- added U$10, U$4, U$5, U$9: VP0550L, transistor-fet:TO92L
- added U$11, U$12, U$6: VN0550L, transistor-fet:TO92L
- added U$13, U$7, U$8: DA-2320, trafo:DIL06
- added X4: BU-SMA-V, con-coax:BU-SMA-V
- C1, C10, C15, C4: value 1n -> .22u; device rcl:C102-043X133 -> resistor:C050-055X075
- C11, C16, C2: value 10p -> .22u; device rcl:C102-043X133 -> resistor:C050-055X075
- C12, C3: value .01u -> .22u; device rcl:C102-043X133 -> resistor:C050-055X075
- C14, C5, C6: value 1u -> .22u; device rcl:C275-205X316 -> resistor:C050-055X075
- C7: value 10p -> (none); device rcl:C102-043X133 -> rcl:C050-030X075
- C8: value .01u -> 10p; device rcl:C102-043X133 -> resistor:C102-064X133
- C9: value 1u -> 10p; device rcl:C275-205X316 -> resistor:C102-064X133
- D1, D4: value 1N4004 -> P6KEXXA; device diode:DO41-10 -> diode:C1702-15
- D2: value 1N4004 -> 4742; device diode:DO41-10 -> diode:ZDIO-10
- D3: value 1N4004 -> 1N4148DO35-10; device diode:DO41-10 -> diode:DO35-10
- R1: value 2M -> 50k; device resistor:P0613/15 -> rcl:0207/10
- R2, R3, R5: value (none) -> 50k; device pot:SP19L -> rcl:0207/10
- R4, R7: value 2M -> 1M; device resistor:P0613/15 -> rcl:0207/10
- U$1: value EMCO-F104PIN -> DA-2320; device dc-dc-converter:EMCO-F -> trafo:DIL06
- U$2: value EMCO-F104PIN -> VN0550L; device dc-dc-converter:EMCO-F -> transistor-fet:TO92L
- U$3: value EMCO-F20CT -> UCC27425; device dc-dc-converter:EMCO-F*CT -> texas:DIL08
- moved C14 209.8 mm to (17.5, -69.8), turned to 0 degrees
- moved C15 202.2 mm to (25.4, -69.8), turned to 0 degrees
- moved C16 196.7 mm to (33.3, -69.8), turned to 0 degrees
- moved C10 138.4 mm to (4.06, -17.0), turned to 0 degrees
- moved C11 137.5 mm to (11.9, -17.0), turned to 0 degrees
- moved C7 123.4 mm to (6.86, 83.3)
- moved C3 121.5 mm to (35.1, 48.5)
- moved C2 116.8 mm to (48.0, 36.3)
- moved C5 110.8 mm to (49.5, 73.9)
- moved D2 101.6 mm to (56.4, 69.3)
- moved C9 98.8 mm to (55.6, 7.87), turned to 180 degrees
- moved C1 97.9 mm to (47.5, 64.3), turned to 0 degrees
- moved C4 94.7 mm to (21.8, 21.8)
- moved R5 93.1 mm to (66.3, 23.6), turned to 270 degrees
- moved D3 93.0 mm to (61.5, 61.2), turned to 180 degrees
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Connections:
- new net +15V: C7.1, D11.C, K1.1, K1.8, K1.9, POWERGD.1, U$3.6
- new net ENSW: CONTROLGD1.1, D11.A, K1.16
- new net N$11: D12.A, R12.2, R5.1, U$6.2
- new net N$16: C5.2, D5.A, D7.A, R8.1
- new net N$17: C8.1, D1.C, D5.C, HV1.TP, R2.2, R4.2, U$1.4, U$4.3
- new net N$18: D1.A, D2.C, D9.C, R1.2, R4.1, R7.2, U$1.5, U$4.1, U$5.3
- new net N$19: C3.2, R13.2
- new net N$20: C4.2, R14.2
- new net N$22: C2.1, U$7.2
- new net N$23: C6.1, U$7.3
- new net N$24: C9.1, D14.A, D4.A, HV2.TP, R11.1, R5.2, U$6.3, U$7.4
- new net N$25: C2.2, D6.C, D8.C, R9.1
- new net N$251: D8.A, R3.1, R9.2, U$2.2
- new net N$26: D15.A, D21.C, OUT.TP, R16.1, R22.2, U$10.1, U$11.1
- new net N$27: C6.2, D12.C, D14.C, R12.1
- new net N$28: C10.1, U$8.2
- new net N$29: C12.1, U$8.3
- new net N$30: C12.2, D17.A, D19.A, R20.1
- new net N$32: D13.C, D17.C, D9.A, R15.2, R18.2, R7.1, U$5.1, U$8.4, U$9.3
- new net N$33: D13.A, D15.C, D16.C, R15.1, R16.2, R17.2, U$10.3, U$8.5, U$9.1
- new net N$34: D18.C, R17.1, R19.2, U$10.2
- new net N$35: C10.2, D16.A, D18.A, R19.1
- new net N$36: D19.C, R18.1, R20.2, U$9.2
- new net N$37: R21.1, U$8.1
- new net N$38: C11.2, R21.2
- new net N$40: C15.1, U$13.2
- new net N$41: C16.1, U$13.3
- new net N$42: C15.2, D22.C, D24.C, R26.1
- new net N$43: C16.2, D23.C, D25.C, R27.1
- new net N$45: U$13.5
- new net N$46: D20.C, D21.A, D22.A, R22.1, R23.2, R24.2, U$11.3, U$12.1
- new net N$47: D25.A, R25.1, R27.2, U$12.2
- new net N$48: R28.1, U$13.1
- new net N$49: C14.2, R28.2
- new net N$50: D24.A, R24.1, R26.2, U$11.2
- new net N$51: D10.C, D20.A, D23.A, R10.2, R23.1, R25.2, U$12.3, U$13.4, U$2.1
- net GND: now also CONTROLGD1.2, K1.11, K1.6, POWERGD.2, U$1.6, U$13.6, U$3.3, U$7.6, U$8.6, X4.2, X4.3, X4.4, X4.5; no longer C1.2, C10.2, C11.2, C12.2, C13.2, C14.2, C15.2, C16.2, C17.2, C18.2, C19.2, C2.2, C3.2, C4.2, C5.2, C6.2, CONTROLHV.4, FDBKHV.4, R2.E, R2.S, R3.E, R3.S, R5.E, R5.S, U$1.P$2, U$1.P$4, U$2.P$2, U$2.P$3, U$3.P$2, U$3.P$5
- net N$1: now also U$3.2, U$3.4, X4.1; no longer C1.1, C2.1, C3.1, C5.1, D1.A, R1.1, U$1.P$3
- net N$10: now also C1.2, D2.A, D3.A, R6.1; no longer C13.1, C14.1, C15.1, C16.1, D4.C, U$3.P$4
- net N$12: now also D7.C, R2.1, R8.2, U$4.2; no longer D4.A, LV-.TP
- net N$13: now also D10.A, D4.C, D6.A, R10.1, R11.2, R3.2, U$2.3, U$6.1; no longer C17.1, CONTROLHV.1, U$1.P$1
- net N$14: now also K1.4, U$3.1; no longer C19.1, CONTROLHV.2, U$3.P$1
- net N$15: now also K1.13, U$3.8; no longer C18.1, CONTROLHV.3, U$2.P$1
- net N$2: now also C11.1, C3.1, U$3.7; no longer C12.1, C4.1, C6.1, C7.1, D2.C, R7.1, U$2.P$4
- net N$3: now also R13.1, U$1.1; no longer FDBKHV.1, R1.2, R2.A
- net N$4: now also C14.1, C4.1, U$3.5; no longer D2.A, HV-.TP
- net N$5: now also C1.1, U$1.2; no longer C10.1, C11.1, C8.1, C9.1, D3.A, R4.1, U$3.P$3
- net N$6: now also R14.1, U$7.1; no longer D1.C, HV+.TP
- net N$7: now also C5.1, U$1.3; no longer FDBKHV.2, R4.2, R5.A
- net N$8: now also D3.C, R1.1, R6.2, U$5.2; no longer FDBKHV.3, R3.A, R7.2
- net N$9: now also U$7.5; no longer D3.C, LV+.TP
Routing:
- net GND: track 493.8 -> 98.9 mm, vias 0 -> 2
- net N$7: track 115.4 -> 10.2 mm, vias 3 -> 0
- net N$3: track 107.9 -> 4.06 mm, vias 2 -> 0
- net N$8: track 118.2 -> 15.7 mm, vias 2 -> 0
- net N$18: track 0.00 -> 101.0 mm
- net N$17: track 0.00 -> 98.4 mm
- net N$24: track 0.00 -> 95.6 mm
- net N$2: track 100.7 -> 20.6 mm
- net +15V: track 0.00 -> 77.6 mm
- net N$10: track 90.6 -> 13.6 mm
- net N$5: track 84.3 -> 10.2 mm
- net N$15: track 84.6 -> 38.1 mm
- net N$1: track 63.0 -> 26.2 mm
- net N$22: track 0.00 -> 21.5 mm
- net N$13: track 87.5 -> 68.3 mm
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Other:
- board size 158.8 x 171.4 mm -> 101.3 x 108 mm

Commit message: two ps in parallel
Parts:
- moved D21 151.5 mm to (91.2, 48.0), turned to 270 degrees
- moved D20 142.2 mm to (96.8, 22.1), turned to 270 degrees
- moved U$12 89.7 mm to (75.4, 13.5)
- moved D13 88.6 mm to (88.1, 4.83), turned to 270 degrees
- moved U$11 85.2 mm to (75.4, -0.25)
- moved U$13 83.1 mm to (41.1, 16.3)
- moved D15 75.1 mm to (98.0, -5.08), turned to 270 degrees
- moved U$10 73.8 mm to (74.9, 45.7)
- moved U$9 73.1 mm to (74.9, 33.5)
- moved C10 65.3 mm to (4.06, -82.3)
- moved C11 65.3 mm to (11.9, -82.3)
- moved C12 65.3 mm to (19.8, -82.3)
- moved C2 65.3 mm to (48.0, -29.0)
- moved C3 65.3 mm to (35.1, -16.8)
- moved C6 65.3 mm to (47.5, -45.2)
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Routing:
- net N$15: track 38.1 -> 103.4 mm
- net N$14: track 38.6 -> 103.9 mm
- net +15V: track 77.6 -> 142.9 mm
- net N$19: track 4.06 -> 69.3 mm
Other:
- board size 101.3 x 108 mm -> 101.3 x 173.2 mm

Commit message: ultra layout. try that next time with lm317 interface
Parts:
- R14, R28: value 1M -> 70
- moved R22 274.0 mm to (96.3, 97.5), turned to 90 degrees
- moved R26 273.4 mm to (75.4, 101.6)
- moved R18 263.9 mm to (80.8, 140.7), turned to 90 degrees
- moved R15 260.2 mm to (97.0, 135.9), turned to 90 degrees
- moved D24 255.9 mm to (75.4, 97.8)
- moved R24 254.7 mm to (80.5, 88.6), turned to 270 degrees
- moved R20 248.6 mm to (75.7, 132.1)
- moved R27 247.0 mm to (75.2, 77.2)
- moved R23 244.7 mm to (96.3, 70.9), turned to 90 degrees
- moved R28 244.1 mm to (48.0, 70.1), turned to 270 degrees
- moved D22 239.3 mm to (70.1, 88.6), turned to 270 degrees
- moved R25 239.1 mm to (80.5, 61.5), turned to 270 degrees
- moved C15 236.0 mm to (62.0, 98.0)
- moved R16 235.4 mm to (97.0, 114.0), turned to 90 degrees
- moved D17 234.7 mm to (70.6, 140.7), turned to 270 degrees
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Routing:
- net GND: track 98.9 -> 224.2 mm, vias 2 -> 1
- net N$51: track 0.00 -> 124.3 mm
- net N$4: track 6.36 -> 105.9 mm, vias 0 -> 1
- net N$33: track 0.00 -> 97.7 mm, vias 0 -> 1
- net N$32: track 0.00 -> 96.9 mm
- net N$46: track 0.00 -> 85.6 mm
- net N$19: track 69.3 -> 6.10 mm
- net N$26: track 0.00 -> 50.6 mm
- net N$15: track 103.4 -> 53.6 mm
- net +15V: track 142.9 -> 94.9 mm
- net N$14: track 103.9 -> 55.9 mm
- net N$2: track 20.6 -> 59.7 mm
- net N$40: track 0.00 -> 20.0 mm
- net N$28: track 0.00 -> 17.3 mm
- net N$34: track 0.00 -> 17.1 mm
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Other:
- board size 101.3 x 173.2 mm -> 115.6 x 201.2 mm
