File: eagle/comboultra.brd (EAGLE design)
At the start: 240 x 164.3 mm, 157 parts, among them IC1 ISO1540, K1 G5V-2, X1 BU-SMA-V, X2 SMA-142-0711-821/826, X3 SMA-142-0711-821/826, X4 BU-SMA-V, X5 SMA-142-0711-821/826, X6 SMA-142-0711-821/826

Commit message: more smd changes
Parts:
- removed C35: 5-20, sprague:SGC3S
- removed C36: 10-30, sprague:SGC3S
- removed C37: 100p, resistor:1111
- removed IC4: (no value), v-reg:317TS
- removed U$16, U$17, U$18, U$19: OPA735DIL, texas:DIL6
- added Q1, Q2, Q3: TIP122V, transistor-npn:TO220V
- C23: value (none) -> 5-20; device resistor:C075-063X106 -> sprague:SGC3S
- C24: value (none) -> 10-30; device resistor:C075-063X106 -> sprague:SGC3S
- C25: value (none) -> 100p; device resistor:C075-063X106 -> resistor:1111
- D1, D10, D13, D15, D20, D21, D4, D9: value P6KEXXA -> SMBJ170D-M3/H; device diode:C1702-15 -> diode:DO214AA
- IC2, IC3: value (none) -> LT1352PA; device v-reg:317TS -> linear-technology:DIL08
- moved C23 103.8 mm to (207.0, 54.0)
- moved C24 101.3 mm to (208.8, 47.9), turned to 270 degrees
- moved C25 95.8 mm to (208.7, 42.7), turned to 0 degrees
- moved X3 77.6 mm to (207.0, 134.2)
- moved L2 77.6 mm to (206.9, 95.5)
- moved TP1 77.6 mm to (210.4, 74.9)
- moved TP3 77.6 mm to (203.6, 75.1)
- moved C27 73.7 mm to (208.8, 120.3)
- moved C28 73.7 mm to (208.7, 115.1)
- moved C26 73.7 mm to (207.0, 126.4)
- moved X5 72.4 mm to (219.7, 61.8)
- moved L3 72.4 mm to (219.6, 23.1)
- moved TP5 72.4 mm to (223.1, 2.54)
- moved TP6 72.4 mm to (216.3, 2.67)
- moved R36 47.4 mm to (154.3, 112.5), turned to 180 degrees
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Connections:
- removed net N$59 (its old number): C20.2, IC3.1, U$18.P$1
- removed net N$62 (its old number): R35.2, R36.1, U$16.P$4
- removed net N$63 (its old number): C21.2, IC4.1, U$17.P$1
- removed net N$68 (its old number): R40.2, U$19.P$3
- new net N$61: C21.2, IC3.1, Q3.1
- new net N$66: IC2.3, R40.2
- new net N$70: CONTROLHV.3, Q3.3
- new net N$71: CONTROLHV.2, Q2.3
- net +12V: now also IC2.8, IC3.8, Q1.2, Q2.2, Q3.2; no longer IC2.3, IC3.3, IC4.3, U$17.P$6, U$18.P$6, U$19.P$6
- net -5V: now also IC2.4, IC3.4; no longer U$16.P$2
- net GND1: now also IC3.5; no longer C23.2, C24.2, C25.2, U$16.P$3, U$17.P$2, U$18.P$2, U$19.P$2
- net N$39: now also IC2.2; no longer U$19.P$4
- net N$44: now also IC3.2, IC3.7; no longer U$16.P$1, U$17.P$4
- net N$45: now also IC2.5; no longer U$18.P$3
- net N$52: now also IC3.3; no longer U$17.P$3
- net N$54: now also Q1.1; no longer U$19.P$1
- net N$56: now also Q1.3; no longer C23.1, IC2.2
- net N$57: now also FDBKHV.2, IC2.6, R38.1; no longer C25.1, CONTROLHV.3, IC4.2
- net N$58: now also C20.2, IC2.7, Q2.1; no longer FDBKHV.2, R38.1, U$18.P$4
- net N$60: now also IC3.6, R35.2, R36.1; no longer C24.1, CONTROLHV.2, IC3.2
- net N$72: now also C23.P$1, C24.P$2, C25.P$1; no longer C26.P$1, C27.P$2, C28.P$1
- net N$73: now also C23.P$2; no longer C26.P$2
- net N$74: now also C24.P$1, C25.P$2; no longer C27.P$1, C28.P$2
- net N$76: now also C26.P$1, C27.P$2, C28.P$1; no longer C29.P$1, C30.P$2, C31.P$1
- net N$77: now also C26.P$2; no longer C29.P$2
- net N$78: now also C27.P$1, C28.P$2; no longer C30.P$1, C31.P$2
- net N$80: now also C29.P$1, C30.P$2, C31.P$1; no longer C32.P$1, C33.P$2, C34.P$1
- net N$81: now also C29.P$2; no longer C32.P$2
- net N$82: now also C30.P$1, C31.P$2; no longer C33.P$1, C34.P$2
- net N$84: now also C32.P$1, C33.P$2, C34.P$1; no longer C35.P$1, C36.P$2, C37.P$1
- net N$85: now also C32.P$2; no longer C35.P$2
- net N$86: now also C33.P$1, C34.P$2; no longer C36.P$1, C37.P$2
- net VCC: no longer U$16.P$6
Routing:
- net N$70: track 0.00 -> 57.2 mm
- net N$39: track 44.3 -> 92.1 mm
- net -5V: track 38.2 -> 85.4 mm, vias 0 -> 2
- net N$61: track 0.00 -> 43.9 mm
- net VCC: track 160.2 -> 130.4 mm
- net N$71: track 0.00 -> 28.7 mm
- net N$62 (its old number): track 26.0 -> 0.00 mm
- net GND: track 261.3 -> 236.6 mm
- net N$59 (its old number): track 22.9 -> 0.00 mm
- net N$63 (its old number): track 22.9 -> 0.00 mm
- net N$57: track 77.3 -> 56.6 mm
- net N$44: track 53.0 -> 33.2 mm
- net N$32: track 87.3 -> 104.9 mm, vias 0 -> 2
- net N$66: track 0.00 -> 17.2 mm
- net N$68 (its old number): track 16.5 -> 0.00 mm
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Other:
- board size 240 x 164.3 mm -> 224.8 x 165.1 mm

Commit message: submit smd board
Parts:
- removed C29, C32: 5-20, sprague:SGC3S
- removed C30, C33: 10-30, sprague:SGC3S
- removed C31, C34: 100p, resistor:1111
- removed L3, L4: B82111, inductors:SUKW1-30
- removed TP5, TP6, TP7, TP8: TPPAD1-13Y, testpad:P1-13Y
- removed X5, X6: SMA-142-0711-821/826, con-coax:J502-ND-142-0711-821/826
- added GND, GND15: TPPAD1-20Y, testpad:P1-20Y
- moved C23 2.54 mm to (209.6, 54.0)
- moved C26 2.54 mm to (209.6, 126.4)
- moved TP1 2.54 mm to (213.0, 74.9)
- moved TP2 2.54 mm to (213.0, 2.54)
- moved TP3 2.54 mm to (206.1, 75.1)
- moved TP4 2.54 mm to (206.1, 2.67)
- moved X2 2.54 mm to (209.6, 61.8)
- moved X3 2.54 mm to (209.6, 134.2)
- moved C24 2.54 mm to (211.3, 47.9)
- moved C25 2.54 mm to (211.2, 42.7)
- moved C27 2.54 mm to (211.3, 120.3)
- moved C28 2.54 mm to (211.2, 115.1)
- moved L1 2.54 mm to (209.4, 23.1)
- moved L2 2.54 mm to (209.4, 95.5)
- moved C13 1.27 mm to (192.0, 58.3)
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Connections:
- removed net N$80: C29.P$1, C30.P$2, C31.P$1, L3.1
- removed net N$81: C29.P$2, X5.1
- removed net N$82: C30.P$1, C31.P$2, TP5.TP, X5.G@1, X5.G@2, X5.G@3, X5.G@4
- removed net N$83: L3.2, TP6.TP
- removed net N$84: C32.P$1, C33.P$2, C34.P$1, L4.1
- removed net N$85: C32.P$2, X6.1
- removed net N$86: C33.P$1, C34.P$2, TP7.TP, X6.G@1, X6.G@2, X6.G@3, X6.G@4
- removed net N$87: L4.2, TP8.TP
- net GND: now also GND.TP, GND15.TP
Routing:
- net N$86: track 57.3 -> 0.00 mm
- net N$82: track 57.3 -> 0.00 mm
- net GND: track 236.6 -> 260.8 mm
- net N$84: track 13.9 -> 0.00 mm
- net N$80: track 13.9 -> 0.00 mm
- net N$83: track 6.57 -> 0.00 mm
- net N$87: track 6.57 -> 0.00 mm
- net N$85: track 3.98 -> 0.00 mm
- net N$81: track 3.98 -> 0.00 mm
Other:
- board size 224.8 x 165.1 mm -> 214.6 x 165.1 mm
