File: eagle/interface_dac_sma_feedback_3PS_LM317_ADC_detector.brd (EAGLE design)
At the start: 112.3 x 143.4 mm, 46 parts, among them IC1 ISO1540, IC2 LT1352PA, IC3 LT1352PA, IC4 LM317MABDT, IC5 LM317MABDT, IC6 LM317MABDT, Q1 TIP122V, Q2 TIP122V, Q3 TIP122V, X1 BU-SMA-V

Commit message: code changes for better safety
Parts:
- removed OK3, OK4: PC817, optocoupler:DIL04
- OK1: value PC817 -> PS2501"; device optocoupler:DIL04 -> optocoupler:DIL16
- moved OK1 25.2 mm to (-18.5, -25.8)
Connections:
- net D7: now also OK1.5; no longer OK4.1
- net D8: now also OK1.3; no longer OK3.1
- net ENSW2: now also OK1.16; no longer OK1.4
- net GND: now also OK1.11, OK1.13, OK1.15; no longer OK1.3, OK3.3, OK4.3
- net N$2: now also OK1.4; no longer OK3.2
- net N$6: now also OK1.6; no longer OK4.2
- net RESET: now also OK1.12; no longer OK4.4
- net SAMPLE: now also OK1.14; no longer OK3.4
Changed lines of the file:
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@@
 <attribute name="OC_FARNELL" value="unknown" x="9.525" y="-5.207" size="1.778" layer="27" display="off"/>
-</element>
-<element name="OK1" library="optocoupler" package="DIL04" value="PC817" x="-7.493" y="-3.175">
-<attribute name="OC_NEWARK" value="97K7059" x="-7.493" y="-3.175" size="1.778" layer="27" display="off"/>
-<attribute name="MPN" value="PC817X4J000F" x="-7.493" y="-3.175" size="1.778" layer="27" display="off"/>
-<attribute name="MF" value="" x="-7.493" y="-3.175" size="1.778" layer="27" display="off"/>
-<attribute name="OC_FARNELL" value="9707727" x="-7.493" y="-3.175" size="1.778" layer="27" display="off"/>
-</element>
-<element name="OK3" library="optocoupler" package="DIL04" value="PC817" x="-16.891" y="-3.175">
-<attribute name="OC_NEWARK" value="97K7059" x="-16.891" y="-3.175" size="1.778" layer="27" display="off"/>
-<attribute name="MPN" value="PC817X4J000F" x="-16.891" y="-3.175" size="1.778" layer="27" display="off"/>
-<attribute name="MF" value="" x="-16.891" y="-3.175" size="1.778" layer="27" display="off"/>
-<attribute name="OC_FARNELL" value="9707727" x="-16.891" y="-3.175" size="1.778" layer="27" display="off"/>
-</element>
-<element name="OK4" library="optocoupler" package="DIL04" value="PC817" x="-26.289" y="-3.175">
-<attribute name="OC_NEWARK" value="97K7059" x="-26.289" y="-3.175" size="1.778" layer="27" display="off"/>
-<attribute name="MPN" value="PC817X4J000F" x="-26.289" y="-3.175" size="1.778" layer="27" display="off"/>
-<attribute name="MF" value="" x="-26.289" y="-3.175" size="1.778" layer="27" display="off"/>
-<attribute name="OC_FARNELL" value="9707727" x="-26.289" y="-3.175" size="1.778" layer="27" display="off"/>
 </element>
 <element name="R14" library="rcl" package="0207/12" value="100" x="-23.495" y="-13.335"/>
 <element name="R15" library="rcl" package="0207/12" value="100" x="-23.495" y="-17.653"/>
+<element name="OK1" library="optocoupler" package="DIL16" value="PS2501&quot;" x="-18.542" y="-25.781"/>
 </elements>
 <signals>
@@
 <contactref element="U$3" pad="3"/>
 <contactref element="U$3" pad="1"/>
-<contactref element="OK1" pad="3"/>
 <contactref element="DATA" pad="3"/>
-<contactref element="OK3" pad="3"/>
-<contactref element="OK4" pad="3"/>
+<contactref element="OK1" pad="15"/>
+<contactref element="OK1" pad="13"/>
+<contactref element="OK1" pad="11"/>
 <wire x1="90.043" y1="110.871" x2="104.013" y2="111.2" width="0" layer="19" extent="1-1"/>
 <wire x1="64.897" y1="107.188" x2="90.043" y2="110.871" width="0" layer="19" extent="1-1"/>
@@
 <wire x1="70.456" y1="136.271" x2="64.897" y2="107.188" width="0" layer="19" extent="1-1"/>
 <wire x1="40.103" y1="136.017" x2="70.456" y2="136.271" width="0" layer="19" extent="1-1"/>
-<wire x1="-6.223" y1="0.635" x2="23.749" y2="63.246" width="0" layer="19" extent="1-1"/>
-<wire x1="-15.621" y1="0.635" x2="-6.223" y2="0.635" width="0" layer="19" extent="1-1"/>
-<wire x1="-25.019" y1="0.635" x2="-15.621" y2="0.635" width="0" layer="19" extent="1-1"/>
-<wire x1="9.525" y1="-5.207" x2="-6.223" y2="0.635" width="0" layer="19" extent="1-1"/>
+<wire x1="9.525" y1="-5.207" x2="23.749" y2="63.246" width="0" layer="19" extent="1-1"/>
+<wire x1="-14.732" y1="-21.971" x2="9.525" y2="-5.207" width="0" layer="19" extent="1-1"/>
+<wire x1="-19.812" y1="-21.971" x2="-14.732" y2="-21.971" width="0" layer="19" extent="1-1"/>
+<wire x1="-24.892" y1="-21.971" x2="-19.812" y2="-21.971" width="0" layer="19" extent="1-1"/>
 </signal>
 <signal name="PWM6">
@@
 <signal name="D7">
 <contactref element="PCB1" pad="D7"/>
-<contactref element="OK4" pad="1"/>
-<wire x1="-27.559" y1="-6.985" x2="38.354" y2="22.479" width="0" layer="19" extent="1-1"/>
+<contactref element="OK1" pad="5"/>
+<wire x1="-17.272" y1="-29.591" x2="38.354" y2="22.479" width="0" layer="19" extent="1-1"/>
 </signal>
 <signal name="D8">
 <contactref element="PCB1" pad="D8"/>
-<contactref element="OK3" pad="1"/>
-<wire x1="-18.161" y1="-6.985" x2="35.814" y2="22.479" width="0" layer="19" extent="1-1"/>
+<contactref element="OK1" pad="3"/>
+<wire x1="-22.352" y1="-29.591" x2="35.814" y2="22.479" width="0" layer="19" extent="1-1"/>
 </signal>
 <signal name="D4">
@@
 <wire x1="33.274" y1="30.099" x2="33.274" y2="22.479" width="1.4224" layer="16"/>
 <contactref element="OK1" pad="1"/>
-<wire x1="-8.763" y1="-6.985" x2="14.732" y2="30.099" width="0" layer="19" extent="16-16"/>
+<wire x1="14.732" y1="30.099" x2="-27.432" y2="-29.591" width="0" layer="19" extent="16-16"/>
 </signal>
 <signal name="N$12">
@@
 <contactref element="CONTROLGD2" pad="1"/>
 <wire x1="14.605" y1="65.965" x2="14.605" y2="49.149" width="1.4224" layer="16"/>
-<contactref element="OK1" pad="4"/>
-<wire x1="-8.763" y1="0.635" x2="14.605" y2="49.149" width="0" layer="19" extent="16-16"/>
+<contactref element="OK1" pad="16"/>
+<wire x1="-27.432" y1="-21.971" x2="14.605" y2="49.149" width="0" layer="19" extent="16-16"/>
 </signal>
 <signal name="SCL">
@@
 <signal name="SAMPLE">
 <contactref element="DATA" pad="4"/>
-<contactref element="OK3" pad="4"/>
-<wire x1="13.485" y1="-5.207" x2="-18.161" y2="0.635" width="0" layer="19" extent="1-1"/>
+<contactref element="OK1" pad="14"/>
+<wire x1="13.485" y1="-5.207" x2="-22.352" y2="-21.971" width="0" layer="19" extent="1-1"/>
 </signal>
 <signal name="RESET">
 <contactref element="DATA" pad="5"/>
-<contactref element="OK4" pad="4"/>
-<wire x1="17.445" y1="-5.207" x2="-27.559" y2="0.635" width="0" layer="19" extent="1-1"/>
+<contactref element="OK1" pad="12"/>
+<wire x1="17.445" y1="-5.207" x2="-17.272" y2="-21.971" width="0" layer="19" extent="1-1"/>
+</signal>
+<signal name="N$2">
+<contactref element="R14" pad="1"/>
+<contactref element="OK1" pad="4"/>
+<wire x1="-29.845" y1="-13.335" x2="-19.812" y2="-29.591" width="0" layer="19" extent="1-1"/>
+</signal>
+<signal name="N$6">
+<contactref element="R15" pad="1"/>
+<contactref element="OK1" pad="6"/>
+<wire x1="-14.732" y1="-29.591" x2="-29.845" y2="-17.653" width="0" layer="19" extent="1-1"/>
 </signal>
 <signal name="N$7">
+<contactref element="OK1" pad="2"/>
 <contactref element="R18" pad="1"/>
-<contactref element="OK1" pad="2"/>
-<wire x1="-6.223" y1="-6.985" x2="17.272" y2="35.814" width="0" layer="19" extent="1-1"/>
-</signal>
-<signal name="N$2">
-<contactref element="OK3" pad="2"/>
-<contactref element="R14" pad="1"/>
-<wire x1="-15.621" y1="-6.985" x2="-29.845" y2="-13.335" width="0" layer="19" extent="1-1"/>
-</signal>
-<signal name="N$6">
-<contactref element="OK4" pad="2"/>
-<contactref element="R15" pad="1"/>
-<wire x1="-25.019" y1="-6.985" x2="-29.845" y2="-17.653" width="0" layer="19" extent="1-1"/>
+<wire x1="17.272" y1="35.814" x2="-24.892" y2="-29.591" width="0" layer="19" extent="1-1"/>
 </signal>
 </signals>
