File: eagle/interface_dac_sma_feedback_3PS_LM317_ADC_detector.sch (EAGLE design)
At the start: 46 parts, among them IC1 ISO1540, IC2 LT1352PA, IC3 LT1352PA, IC4 LM317MABDT, IC5 LM317MABDT, IC6 LM317MABDT, Q1 TIP122V, Q2 TIP122V, Q3 TIP122V, X1 BU-SMA-V

Commit message: code changes for better safety
Parts:
- removed OK3, OK4: PC817, optocoupler:PC817
- OK1: value PC817 -> PS2501"; device optocoupler:PC817 -> optocoupler:PS2501"
Connections:
- net D7: now also OK1C.A; no longer OK4.A
- net D8: now also OK1B.A; no longer OK3.A
- net ENSW2: now also OK1A.COL; no longer OK1.COL
- net GND: now also OK1A.EMI, OK1B.EMI, OK1C.EMI; no longer OK1.EMIT, OK3.EMIT, OK4.EMIT
- net N$2: now also OK1B.C; no longer OK3.C
- net N$6: now also OK1C.C; no longer OK4.C
- net N$7: now also OK1A.C; no longer OK1.C
- net PWM9: now also OK1A.A; no longer OK1.A
- net RESET: now also OK1C.COL; no longer OK4.COL
- net SAMPLE: now also OK1B.COL; no longer OK3.COL
Other:
- moved on the sheet: OK1A, R14, R15, R18
Changed lines of the file:
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@@
 <part name="GND12" library="supply1" deviceset="GND" device=""/>
 <part name="DATA" library="con-molex" deviceset="KK-156-5" device=""/>
-<part name="OK1" library="optocoupler" deviceset="PC817" device=""/>
-<part name="OK3" library="optocoupler" deviceset="PC817" device=""/>
-<part name="OK4" library="optocoupler" deviceset="PC817" device=""/>
 <part name="GND19" library="supply1" deviceset="GND" device=""/>
 <part name="R14" library="rcl" deviceset="R-US_" device="0207/12" value="100"/>
@@
 <part name="GND21" library="supply1" deviceset="GND" device=""/>
 <part name="GND24" library="supply1" deviceset="GND" device=""/>
+<part name="OK1" library="optocoupler" deviceset="PS2501" device="&quot;"/>
 </parts>
 <sheets>
@@
 <instance part="X1" gate="G$1" x="543.56" y="45.72" rot="R90"/>
 <instance part="GND17" gate="1" x="546.1" y="50.8" rot="R180"/>
-<instance part="R18" gate="G$1" x="322.58" y="45.72" rot="R180"/>
+<instance part="R18" gate="G$1" x="320.04" y="50.8" rot="R180"/>
 <instance part="GND1" gate="1" x="345.44" y="43.18"/>
 <instance part="CONTROLGD2" gate="-1" x="355.6" y="50.8"/>
@@
 <instance part="DATA" gate="-4" x="309.88" y="-27.94"/>
 <instance part="DATA" gate="-5" x="309.88" y="-30.48"/>
-<instance part="OK1" gate="A" x="337.82" y="48.26"/>
-<instance part="OK3" gate="A" x="335.28" y="-38.1"/>
-<instance part="OK4" gate="A" x="335.28" y="-53.34"/>
 <instance part="GND19" gate="1" x="302.26" y="-25.4" rot="R270"/>
-<instance part="R14" gate="G$1" x="320.04" y="-40.64" rot="R180"/>
-<instance part="R15" gate="G$1" x="320.04" y="-55.88" rot="R180"/>
+<instance part="R14" gate="G$1" x="320.04" y="-35.56" rot="R180"/>
+<instance part="R15" gate="G$1" x="320.04" y="-50.8" rot="R180"/>
 <instance part="GND21" gate="1" x="350.52" y="-40.64" rot="R90"/>
 <instance part="GND24" gate="1" x="350.52" y="-55.88" rot="R90"/>
+<instance part="OK1" gate="A" x="337.82" y="48.26"/>
+<instance part="OK1" gate="B" x="335.28" y="-38.1"/>
+<instance part="OK1" gate="C" x="335.28" y="-53.34"/>
 </instances>
 <busses>
@@
 </segment>
 <segment>
-<pinref part="GND1" gate="1" pin="GND"/>
-<pinref part="OK1" gate="A" pin="EMIT"/>
-</segment>
-<segment>
 <pinref part="DATA" gate="-3" pin="S"/>
 <wire x1="307.34" y1="-25.4" x2="304.8" y2="-25.4" width="0.1524" layer="91"/>
@@
 </segment>
 <segment>
-<pinref part="OK3" gate="A" pin="EMIT"/>
 <pinref part="GND21" gate="1" pin="GND"/>
 <wire x1="342.9" y1="-40.64" x2="347.98" y2="-40.64" width="0.1524" layer="91"/>
-</segment>
-<segment>
-<pinref part="OK4" gate="A" pin="EMIT"/>
+<pinref part="OK1" gate="B" pin="EMI"/>
+</segment>
+<segment>
 <pinref part="GND24" gate="1" pin="GND"/>
 <wire x1="342.9" y1="-55.88" x2="347.98" y2="-55.88" width="0.1524" layer="91"/>
+<pinref part="OK1" gate="C" pin="EMI"/>
+</segment>
+<segment>
+<pinref part="GND1" gate="1" pin="GND"/>
+<pinref part="OK1" gate="A" pin="EMI"/>
 </segment>
 </net>
@@
 </segment>
 <segment>
-<pinref part="OK4" gate="A" pin="A"/>
-<wire x1="325.12" y1="-50.8" x2="322.58" y2="-50.8" width="0.1524" layer="91"/>
-<label x="325.12" y="-48.26" size="1.778" layer="95" rot="R180"/>
+<wire x1="325.12" y1="-55.88" x2="322.58" y2="-55.88" width="0.1524" layer="91"/>
+<label x="322.58" y="-55.88" size="1.778" layer="95" rot="R180"/>
+<pinref part="OK1" gate="C" pin="A"/>
 </segment>
 </net>
@@
 </segment>
 <segment>
-<pinref part="OK3" gate="A" pin="A"/>
-<wire x1="325.12" y1="-35.56" x2="322.58" y2="-35.56" width="0.1524" layer="91"/>
-<label x="325.12" y="-33.02" size="1.778" layer="95" rot="R180"/>
+<wire x1="325.12" y1="-40.64" x2="322.58" y2="-40.64" width="0.1524" layer="91"/>
+<label x="322.58" y="-40.64" size="1.778" layer="95" rot="R180"/>
+<pinref part="OK1" gate="B" pin="A"/>
 </segment>
 </net>
@@
 <net name="AGND" class="0">
 <segment>
-<wire x1="304.8" y1="45.72" x2="317.5" y2="45.72" width="0.1524" layer="91"/>
+<wire x1="312.42" y1="50.8" x2="314.96" y2="50.8" width="0.1524" layer="91"/>
 <pinref part="R18" gate="G$1" pin="2"/>
-<label x="304.8" y="45.72" size="1.778" layer="95" rot="R180"/>
+<label x="302.26" y="53.34" size="1.778" layer="95" rot="R180"/>
 </segment>
 <segment>
@@
 </segment>
 <segment>
-<wire x1="309.88" y1="-40.64" x2="314.96" y2="-40.64" width="0.1524" layer="91"/>
+<wire x1="312.42" y1="-35.56" x2="314.96" y2="-35.56" width="0.1524" layer="91"/>
 <pinref part="R14" gate="G$1" pin="2"/>
-<label x="312.42" y="-40.64" size="1.778" layer="95" rot="R180"/>
-</segment>
-<segment>
-<wire x1="309.88" y1="-55.88" x2="314.96" y2="-55.88" width="0.1524" layer="91"/>
+<label x="312.42" y="-35.56" size="1.778" layer="95" rot="R180"/>
+</segment>
+<segment>
+<wire x1="309.88" y1="-50.8" x2="314.96" y2="-50.8" width="0.1524" layer="91"/>
 <pinref part="R15" gate="G$1" pin="2"/>
-<label x="312.42" y="-55.88" size="1.778" layer="95" rot="R180"/>
+<label x="309.88" y="-50.8" size="1.778" layer="95" rot="R180"/>
 </segment>
 </net>
@@
 </segment>
 <segment>
-<wire x1="327.66" y1="50.8" x2="304.8" y2="50.8" width="0.1524" layer="91"/>
+<label x="304.8" y="45.72" size="1.778" layer="95" rot="R180"/>
 <pinref part="OK1" gate="A" pin="A"/>
-<label x="304.8" y="50.8" size="1.778" layer="95" rot="R180"/>
+<wire x1="327.66" y1="45.72" x2="312.42" y2="45.72" width="0.1524" layer="91"/>
 </segment>
 </net>
@@
 </segment>
 <segment>
-<pinref part="OK3" gate="A" pin="COL"/>
 <wire x1="342.9" y1="-35.56" x2="350.52" y2="-35.56" width="0.1524" layer="91"/>
 <label x="350.52" y="-33.02" size="1.778" layer="95" rot="R180"/>
+<pinref part="OK1" gate="B" pin="COL"/>
 </segment>
 </net>
@@
 </segment>
 <segment>
-<pinref part="OK4" gate="A" pin="COL"/>
 <wire x1="342.9" y1="-50.8" x2="350.52" y2="-50.8" width="0.1524" layer="91"/>
 <label x="350.52" y="-48.26" size="1.778" layer="95" rot="R180"/>
+<pinref part="OK1" gate="C" pin="COL"/>
+</segment>
+</net>
+<net name="N$2" class="0">
+<segment>
+<pinref part="R14" gate="G$1" pin="1"/>
+<pinref part="OK1" gate="B" pin="C"/>
+</segment>
+</net>
+<net name="N$6" class="0">
+<segment>
+<pinref part="R15" gate="G$1" pin="1"/>
+<pinref part="OK1" gate="C" pin="C"/>
 </segment>
 </net>
 <net name="N$7" class="0">
 <segment>
+<pinref part="OK1" gate="A" pin="C"/>
 <pinref part="R18" gate="G$1" pin="1"/>
-<pinref part="OK1" gate="A" pin="C"/>
-</segment>
-</net>
-<net name="N$2" class="0">
-<segment>
-<pinref part="OK3" gate="A" pin="C"/>
-<pinref part="R14" gate="G$1" pin="1"/>
-</segment>
-</net>
-<net name="N$6" class="0">
-<segment>
-<pinref part="OK4" gate="A" pin="C"/>
-<pinref part="R15" gate="G$1" pin="1"/>
-</segment>
-</net>
+<wire x1="325.12" y1="50.8" x2="327.66" y2="50.8" width="0.1524" layer="91"/>
+</segment>
+</net>
