File: eagle/hv_lv_combo.brd (EAGLE design)
At the start: 158.8 x 119.4 mm, 22 parts

Commit message: update for thermal issues and CTIA breakout
Parts:
- added C10, C13: 1n, rcl:C102-043X133
- added C11, C14: 10p, rcl:C102-043X133
- added C8, C9: 1u, rcl:C275-205X316
- added J1, J2: PIN2F061.100, con-faston:F061.100
- added POWERDETECT, POWERIFACE: (no value), con-molex:KK-156-4
- added POWERGD, POWERGD1: (no value), con-molex:KK-156-2
- added R4: (no value), pot:SP19L
- added U$3: IRM-30-15, meanwell:IRM-30-15
- added U$4, U$5: EMCO-F104PIN, dc-dc-converter:EMCO-F
- C1: value 1n -> (none); device rcl:C102-043X133 -> rcl:E5-13
- C2: value 10p -> (none); device rcl:C102-043X133 -> rcl:E5-13
- C3: value .01u -> (none); device rcl:C102-043X133 -> rcl:C050-050X075
- C4: value 1n -> (none); device rcl:C102-043X133 -> rcl:C050-050X075
- C5: value 1u -> (none); device rcl:C275-205X316 -> rcl:C050-050X075
- C6: value 1u -> (none); device rcl:C275-205X316 -> rcl:E5-13
- C7: value 10p -> .01u
- R1: value 2M -> VARISTOR-7,5; device resistor:P0613/15 -> varistor:R-7,5
- R2: value (none) -> 2M; device pot:SP19L -> resistor:P0613/15
- U$1: value EMCO-F104PIN -> IRM-05-05; device dc-dc-converter:EMCO-F -> meanwell:IRM-05-05
- U$2: value EMCO-F104PIN -> IRM-60-12; device dc-dc-converter:EMCO-F -> meanwell:IRM-60-12
- moved HV- 232.9 mm to (103.9, 279.1), turned to 270 degrees
- moved D2 219.9 mm to (85.9, 279.1), turned to 0 degrees
- moved C7 208.7 mm to (33.3, 246.1), turned to 180 degrees
- moved HV+ 187.7 mm to (46.0, 270.3), turned to 180 degrees
- moved C12 179.1 mm to (103.1, 230.9), turned to 0 degrees
- moved R3 174.2 mm to (13.0, 238.0)
- moved R7 169.7 mm to (85.9, 237.2), turned to 180 degrees
- moved D1 168.6 mm to (46.0, 256.3), turned to 270 degrees
- moved R2 118.0 mm to (30.7, 229.6), turned to 180 degrees
- moved R1 116.7 mm to (10.4, 51.1), turned to 0 degrees
- moved C5 115.8 mm to (113.8, 16.3), turned to 270 degrees
- moved C18 105.5 mm to (87.9, 144.8), turned to 180 degrees
- moved U$2 90.3 mm to (99.8, 123.2), turned to 180 degrees
- moved U$1 78.7 mm to (30.0, 42.9)
- moved C2 69.7 mm to (92.7, 53.3)
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Connections:
- removed net N$3: FDBKHV.1, R1.2, R2.A
- new net +15V: C1.+, C4.1, POWERDETECT.1, POWERGD.1, POWERIFACE.1, U$2.P$1
- new net -15V: C5.2, C6.-, POWERDETECT.4, POWERIFACE.4, U$3.-V
- new net GND1: C10.2, C11.2, C12.2, C13.2, C14.2, C17.2, C18.2, C7.2, C8.2, C9.2, CONTROLHV.2, FDBKHV.2, R3.E, R3.S, R4.E, R4.S, U$4.P$2, U$4.P$4, U$5.P$2, U$5.P$3
- new net N$4: C10.1, C11.1, C7.1, C8.1, D1.A, R2.1, U$4.P$3
- new net N$5: C12.1, C13.1, C14.1, C9.1, D2.C, R7.1, U$5.P$4
- new net N$6: FDBKHV.1, R2.2, R3.A
- new net VCC: C2.+, C3.1, POWERDETECT.2, POWERGD1.1, POWERIFACE.2, U$1.+V
- net GND: now also C1.-, C2.-, C5.1, C6.+, POWERDETECT.3, POWERGD.2, POWERGD1.2, POWERIFACE.3, U$1.-V, U$3.+V; no longer C1.2, C12.2, C17.2, C18.2, C2.2, C5.2, C6.2, C7.2, CONTROLHV.2, FDBKHV.2, R2.E, R2.S, R3.E, R3.S, U$1.P$2, U$1.P$4, U$2.P$3
- net N$1: now also J1.A1, J1.A2, R1.2, U$1.ACN, U$2.P$4, U$3.ACN; no longer C1.1, C2.1, C3.1, C5.1, D1.A, R1.1, U$1.P$3
- net N$13: now also U$4.P$1; no longer U$1.P$1
- net N$15: now also U$5.P$1; no longer U$2.P$1
- net N$2: now also J2.A1, J2.A2, R1.1, U$1.ACL, U$2.P$3, U$3.ACL; no longer C12.1, C4.1, C6.1, C7.1, D2.C, R7.1, U$2.P$4
- net N$8: now also R4.A; no longer R3.A
Routing:
- net GND: track 299.7 -> 0.00 mm
- net GND1: track 0.00 -> 299.7 mm
- net +15V: track 0.00 -> 105.8 mm
- net N$6: track 0.00 -> 96.1 mm
- net N$3: track 96.1 -> 0.00 mm
- net VCC: track 0.00 -> 92.0 mm
- net N$5: track 0.00 -> 91.8 mm
- net N$1: track 63.0 -> 127.5 mm
- net N$4: track 0.00 -> 63.0 mm
- net -15V: track 0.00 -> 60.5 mm
- net N$2: track 91.8 -> 121.8 mm
- added copper zone on layer 16, net GND1
- added copper zone on layer 16, net N$3
Other:
- board size 158.8 x 119.4 mm -> 123.4 x 286.5 mm
