File: eagle/gdctia.brd (EAGLE design)
At the start: 101.9 x 165.1 mm, 98 parts, among them K1 G5V-2, X4 BU-SMA-V

Commit message: gd mods
Parts:
- added C13, C17, C4: 10n, rcl:C050-050X075
- added IC1: IVC102UADAPTOR, burr-brown:DIL14
- added IC2: LT1352PA, linear-technology:DIL08
- added IC3: AD580H, linear:TO39
- added R38, R39: 10k, resistor:0207/15
- added R40, R43: 10k, resistor:0207/10
- added R41, R42: 1.5M, resistor:0207/10
- added SW2: (no value), special:EDG-03
- added U$22, U$31: CTIA, ctia:CTIA
- added U$23, U$24, U$25, U$30: VP2450, transistor-fet:SOT89-BCE
- added U$26, U$27, U$28, U$29: VN2450, transistor-fet:SOT89-BCE
- added X1: 1-227161-0, con-coax:AMP_227161
- added X5: (no value), con-subd:F09HP
- moved C3 17.8 mm to (116.1, 102.1)
- moved HV1 17.8 mm to (105.4, 159.3)
- moved HV2 17.8 mm to (105.7, 7.87)
- moved OUT 17.8 mm to (116.1, 81.3)
- moved R10 17.8 mm to (104.6, 35.1)
- moved R11 17.8 mm to (104.6, 17.3)
- moved R15 17.8 mm to (101.9, 110.2)
- moved R16 17.8 mm to (101.9, 90.7)
- moved R22 17.8 mm to (101.9, 67.6)
- moved R23 17.8 mm to (104.6, 50.3)
- moved R33 17.8 mm to (97.8, 121.2)
- moved R35 17.8 mm to (115.8, 70.9)
- moved R36 17.8 mm to (115.8, 57.9)
- moved R37 17.8 mm to (116.1, 93.0)
- moved R4 17.8 mm to (102.1, 146.1)
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Connections:
- new net +15V1: C13.1, IC1.14, IC2.8, X5.1
- new net +5V: C17.1, IC3.1, R38.1, R39.1, X5.5
- new net -15V: C4.1, IC1.9, IC2.4, X5.4
- new net GND1: C17.2, C4.2, IC1.1, IC1.13, IC3.3, R43.1, X5.2, X5.3, X5.9
- new net GND2: X1.2
- new net N$58: IC1.6, SW2.1
- new net N$59: IC1.5, SW2.2
- new net N$60: IC1.4, SW2.3
- new net N$61: IC1.3, SW2.4, SW2.5, SW2.6
- new net N$62: IC1.10, R40.2
- new net N$63: IC2.2, R40.1, R41.2
- new net N$64: IC2.3, R42.1, R43.2
- new net N$65: IC3.2, R42.2
- new net N$66: U$31.P$1, X1.1
- new net RESET: IC1.12, R39.2, X5.6
- new net SAMPLE: IC1.11, R38.2, X5.7
- new net VIN: IC1.2, U$22.P$1
- new net VOUT: IC2.1, R41.1, X5.8
- net N$11: now also U$29.B
- net N$12: now also U$25.B
- net N$13: now also U$29.C, U$29.C@1
- net N$18: now also U$25.C, U$25.C@1
- net N$19: now also U$26.E
- net N$20: now also U$25.E
- net N$21: now also U$24.E
- net N$251: now also U$28.B
- net N$26: now also U$26.C, U$26.C@1, U$30.C, U$30.C@1
- net N$3: now also U$29.E
- net N$31: now also U$30.E
- net N$32: now also U$24.C, U$24.C@1
- net N$33: now also U$23.C, U$23.C@1
- net N$34: now also U$30.B
- net N$36: now also U$23.B
- net N$39: now also U$23.E
- net N$46: now also U$27.C, U$27.C@1
- net N$47: now also U$27.B
- net N$50: now also U$26.B
- net N$51: now also U$28.C, U$28.C@1
- net N$6: now also U$28.E
- net N$8: now also U$24.B
- net N$9: now also U$27.E
Routing:
- net +15V1: track 0.00 -> 107.0 mm
- net +5V: track 0.00 -> 69.7 mm
- net -15V: track 0.00 -> 63.6 mm, vias 0 -> 1
- net RESET: track 0.00 -> 58.2 mm
- net SAMPLE: track 0.00 -> 58.1 mm
- net N$32: track 87.9 -> 144.7 mm
- net N$26: track 61.7 -> 103.7 mm
- net N$64: track 0.00 -> 41.6 mm, vias 0 -> 2
- net N$33: track 80.4 -> 121.2 mm
- net N$18: track 100.9 -> 139.0 mm
- net GND: track 390.2 -> 427.5 mm
- net N$13: track 68.6 -> 105.5 mm
- net N$46: track 64.9 -> 101.1 mm
- net N$17: track 76.5 -> 111.0 mm
- net VIN: track 0.00 -> 33.7 mm
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- added copper zone on layer 16, net GND1
- added copper zone on layer 16, net GND2
Other:
- board size 101.9 x 165.1 mm -> 217.9 x 165.1 mm
