File: eagle/hvreg_feedback_2PS.sch (EAGLE design)
At the start: 22 parts

Commit message: Square wave one side/dc other
Connections:
- net GND: now also U$2.+VOUT; no longer U$2.-VOUT
- net N$2: now also D2.C, U$2.-VOUT; no longer D2.A, U$2.+VOUT
- net N$4: now also D2.A; no longer D2.C
Other:
- moved on the sheet: C18, CONTROLHV-3, D2, U$2
