File: eagle/interface_dac_sma_feedback_2PS_ADC_detector_SMD.sch (EAGLE design)
At the start: 106 parts, among them K1 G5V-2, X4 BU-SMA-V

Commit message: Square wave one side/dc other
Parts:
- removed C10, C11, C12, C14, C15, C16: 1u, resistor:C-USC0805
- removed C8, C9: 10p, resistor:C-US102-064X133
- removed CONTROLGD1, POWERGD: (no value), con-molex:KK-156-2
- removed D11: 1N4148DO35-10, diode:1N4148DO35-10
- removed D12, D18, D19, D24, D25, D3, D7, D8: (no value), diode:DIODE-SMB
- removed D14, D16, D17, D2, D22, D23, D5, D6: 1SMB5918BT3G, diode:ZENER-DIODESMB
- removed GND, GND15, HV1, HV2, OUT: TPPAD1-20Y, testpad:TPPAD1-20Y
- removed K1: G5V-2, relay:G5V-2
- removed R11, R22, R23, R35, R36, R37, R4: 10M, rcl:R-US_R2512
- removed R17, R24, R25: 100k, rcl:R-US_R0805
- removed R19, R20, R21, R26, R27, R28: 10, rcl:R-US_R0805
- removed R29, R30: 6.67, rcl:R-US_R0805
- removed R31, R32, R33, R34: 1.25, rcl:R-US_R0805
- removed U$10, U$4, U$5, U$9: VP0550L, transistor-fet:VP0550L
- removed U$11, U$12, U$6: VN0550L, transistor-fet:VN0550L
- removed U$13, U$7, U$8: DA-2320SMD6, trafo:DA-2320SMD6
- removed U$14, U$15, U$16, U$17, U$18, U$19, U$20, U$21: SMBJ170D-M3/H, diode:SMBJ170D-M3/H
- removed U$23, U$24, U$25, U$30: VP2450, transistor-fet:VP2450
- removed U$26, U$27, U$28, U$29: VN2450, transistor-fet:VN2450
- removed X4: BU-SMA-V, con-coax:BU-SMA-V
- added C4: 10n, resistor:C-USC0805
- added CONTROLGD2: (no value), con-molex:KK-156-2
- added CONTROLHV, FDBKHV: (no value), con-molex:KK-156-3
- added CTIA, POWERINTERFACE: (no value), con-molex:KK-156-4
- added IC1: ISO1540SMD, texas:ISO1540SMD
- added IC2, IC3: LT1352SA, linear-technology:LT1352SA
- added OK1: PS2501", optocoupler:PS2501"
- added PCB1: ARDUINO_MICRO, E14_Arduino_published:ARDUINO_MICRO
- added Q1, Q2: 2N3055, transistor-npn:2N3055
- added X1: BU-SMA-V, con-coax:BU-SMA-V
- C1: value 1u -> 10n; device resistor:C-USC0805 -> rcl:C-USC0805
- C2, C5, C6: value 1u -> 10n
- C7: device rcl:C-US050-030X075 -> resistor:C-USC0805
- R1, R2, R3: value 100k -> 10k; device rcl:R-US_R0805 -> resistor:R-US_R0805
- R10: value 10M -> 10k; device rcl:R-US_R2512 -> resistor:R-US_R0805
- R12, R6, R9: value 10 -> 10k; device rcl:R-US_R0805 -> resistor:R-US_R0805
- R13: value 6.67 -> 10k; device rcl:R-US_R0805 -> resistor:R-US_R0805
- R14: value 6.67 -> 100
- R15: value 10M -> 100; device rcl:R-US_R2512 -> rcl:R-US_R0805
- R16: value 10M -> 100k; device rcl:R-US_R2512 -> pot:TRIM_US-B90P
- R18: value 100k -> 100
- R5: value 100k -> 20k; device rcl:R-US_R0805 -> resistor:R-US_R0805
- R7: value 10M -> 40k; device rcl:R-US_R2512 -> resistor:R-US_R0805
- R8: value 10 -> 20k; device rcl:R-US_R0805 -> resistor:R-US_R0805
- U$1: value DA-2320SMD6 -> LTC6992SMD; device trafo:DA-2320SMD6 -> linear-technology:LTC6992SMD
- U$2: value VN0550L -> MCP4728; device transistor-fet:VN0550L -> microchip:MCP4728
- U$3: value UCC27425 -> ADS1015; device texas:UCC27425 -> texas:ADS1015
Connections:
- removed net ENSW: CONTROLGD1-1.S, D11.A, K1A.2
- removed net N$10: C1.2, D2.A, D3.A, R6.1
- removed net N$11: D12.A, R12.2, R5.1, U$29.G, U$6.G
- removed net N$15: K12.P, U$3.ENB
- removed net N$17: C8.1, D5.C, HV1.TP, R2.2, R34.1, R4.2, U$1.3, U$14.C
- removed net N$22: C2.1, U$7.6
- removed net N$251: D8.A, R3.1, R9.2, U$2.G, U$28.G
- removed net N$27: C6.2, D12.C, D14.C, R12.1
- removed net N$28: C10.1, U$8.6
- removed net N$29: C12.1, U$8.4
- removed net N$30: C12.2, D17.A, D19.A, R20.1
- removed net N$31: R31.2, U$10.S, U$30.S
- removed net N$32: D17.C, R15.2, R18.2, R32.1, R7.1, U$24.D, U$5.D, U$8.3
- removed net N$33: D16.C, R15.1, R16.2, R17.2, R31.1, U$23.D, U$8.5, U$9.D
- removed net N$34: D18.C, R17.1, R19.2, U$10.G, U$30.G
- removed net N$35: C10.2, D16.A, D18.A, R19.1
- removed net N$36: D19.C, R18.1, R20.2, U$23.G, U$9.G
- removed net N$37: R21.1, U$1.1, U$8.1
- removed net N$38: C11.2, R21.2
- removed net N$39: R32.2, U$23.S, U$9.S
- removed net N$40: C15.1, U$13.6
- removed net N$41: C16.1, U$13.4
- removed net N$42: C15.2, D22.C, D24.C, R26.1
- removed net N$43: C16.2, D23.C, D25.C, R27.1
- removed net N$44: R35.1, R36.2
- removed net N$45: C3.1, R37.1
- removed net N$46: D22.A, R22.1, R23.2, R24.2, R30.1, U$12.D, U$13.5, U$27.D
- removed net N$47: D25.A, R25.1, R27.2, U$12.G, U$27.G
- removed net N$48: R28.1, U$13.1, U$7.1
- removed net N$49: C14.2, R28.2
- removed net N$50: D24.A, R24.1, R26.2, U$11.G, U$26.G
- removed net N$51: D23.A, R10.2, R23.1, R25.2, R29.1, U$13.3, U$2.D, U$28.D
- removed net N$52: U$14.A, U$15.C
- removed net N$53: U$15.A, U$16.C
- removed net N$54: U$16.A, U$17.C
- removed net N$55: U$18.C, U$19.A
- removed net N$56: U$19.C, U$20.A
- removed net N$57: U$20.C, U$21.A
- removed net N$9: R29.2, U$12.S, U$27.S
- new net -15V: C5.1, IC2A.V-, IC3A.V-, POWERINTERFACE-4.S
- new net A+5: IC1.VCC1, PCB1.+5V
- new net AGND: IC1.GND1, PCB1.GND., R14.2, R15.2, R18.2
- new net CTIA: CTIA-4.S, U$3.AIN1
- new net D10: PCB1.D10
- new net D11: PCB1.D11
- new net D4: PCB1.D4
- new net D7: OK1C.A, PCB1.D7
- new net D8: OK1B.A, PCB1.D8
- new net ENSW2: CONTROLGD2-1.S, OK1A.COL
- new net PWM5: PCB1.D5
- new net PWM6: PCB1.D6
- new net PWM9: OK1A.A, PCB1.D9
- new net RDBK1: FDBKHV-1.S, IC2A.-IN, R3.1, U$3.AIN0
- new net RDBK3: IC3A.-IN, R13.2, R9.1, U$3.AIN2
- new net RDBK4: C2.1, R6.2, R7.2, U$1.P$1, U$3.AIN3
- new net RESET: CTIA-3.S, OK1C.COL
- new net SAMPLE: CTIA-2.S, OK1B.COL
- new net SCL: IC1.SCL1, PCB1.D3
- new net SCL_OUT: IC1.SCL2, R2.1, U$2.SCL, U$3.SCL
- new net SDA: IC1.SDA1, PCB1.D2
- new net SDA_OUT: IC1.SDA2, R1.1, U$2.SDA, U$3.SDA
- new net VCC: C1.1, C4.1, IC1.VCC2, POWERINTERFACE-2.S, R1.2, R2.2, U$1.P$5, U$2.VDD, U$3.VDD
- net +15V: now also IC2A.V+, IC3A.V+, POWERINTERFACE-1.S, Q1.C, Q2.C; no longer D11.C, K11.S, K12.S, K1A.1, POWERGD-1.S, U$3.VCC
- net GND: now also C1.2, C2.2, C4.2, C5.2, CONTROLGD2-2.S, CONTROLHV-2.S, CTIA-1.S, FDBKHV-2.S, IC1.GND2, IC3B.+IN, OK1A.EMI, OK1B.EMI, OK1C.EMI, POWERINTERFACE-3.S, R16.A, R16.S, R6.1, U$1.P$2, U$1.P$4, U$2.VSS, U$2._LDAC, U$3.ADDR, X1.2; no longer C3.2, C8.2, C9.2, CONTROLGD1-2.S, GND.TP, GND15.TP, K11.O, K12.O, POWERGD-2.S, R36.1, U$1.2, U$13.2, U$17.A, U$21.C, U$7.2, U$8.2, X4.2
- net N$1: now also R7.1, U$2.VOUTA; no longer U$3.INA, U$3.INB, X4.1
- net N$12: now also R16.E, U$1.P$3; no longer D7.C, R2.1, R8.2, U$25.G, U$4.G
- net N$13: now also U$1.P$6, X1.1; no longer D6.A, R10.1, R11.2, R14.1, R3.2, U$29.D, U$6.D, U$7.5
- net N$14: now also IC3B.OUT, R13.1, R8.2; no longer K11.P, U$3.ENA
- net N$16: now also IC2A.+IN, R10.2; no longer C5.2, D5.A, D7.A, R8.1
- net N$18: now also IC3A.+IN, R12.2; no longer D2.C, R1.2, R33.1, R4.1, R7.2, U$1.5, U$25.D, U$4.D
- net N$19: now also C3.2, IC2A.OUT, Q1.B; no longer R30.2, U$11.S, U$26.S
- net N$2: now also OK1B.C, R14.1; no longer C11.1, U$3.OUTA
- net N$20: now also C6.1, R9.2; no longer R34.2, U$25.S, U$4.S
- net N$21: now also C6.2, IC3A.OUT, Q2.B; no longer R33.2, U$24.S, U$5.S
- net N$23: now also IC3B.-IN, R5.2, R8.1; no longer C6.1, U$7.4
- net N$24: now also R10.1, U$2.VOUTD; no longer C9.1, D14.A, HV2.TP, R11.1, R13.1, R5.2, U$18.A, U$7.3
- net N$25: now also R12.1, U$2.VOUTB; no longer C2.2, D6.C, D8.C, R9.1
- net N$26: now also U$2.VOUTC; no longer OUT.TP, R16.1, R22.2, R35.2, R37.2, U$10.D, U$11.D, U$26.D, U$30.D
- net N$3: now also C3.1, R3.2; no longer R13.2, U$29.S, U$6.S
- net N$4: now also CONTROLHV-1.S, Q1.E; no longer C14.1, U$3.OUTB
- net N$5: now also CONTROLHV-3.S, Q2.E; no longer C1.1, U$1.6
- net N$6: now also OK1C.C, R15.1; no longer R14.2, U$2.S, U$28.S
- net N$7: now also OK1A.C, R18.1; no longer C5.1, U$1.4
- net N$8: now also FDBKHV-3.S, R5.1; no longer D3.C, R1.1, R6.2, U$24.G, U$5.G
Other:
- moved on the sheet: C1, C2, C3, C5, C6, C7, R1, R10, R12, R13, R14, R15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
