File: eagle/gd_new_combo.brd (EAGLE design)
At the start: 152.7 x 152.4 mm, 56 parts, among them K1 G5V-2, X4 BU-SMA-V

Commit message: timing ctia
Parts:
- added C24, C25, C26, C27, C28, C29: .22u, resistor:C050-055X075
- added C30: (no value), rcl:C050-030X075
- added C31, C32: 10p, resistor:C102-064X133
- added CONTROLGD2, POWERGD1: (no value), con-molex:KK-156-2
- added D10, D12, D13, D14: P6KEXXA, diode:C1702-15
- added D15, D16, D17, D18: 4742, diode:ZDIO-10
- added D19, D20, D21, D22, D9: 1N4148DO35-10, diode:DO35-10
- added GND1, GND13, HV1, HV2, OUT1: TPPAD1-20Y, testpad:P1-20Y
- added K2: G5V-2, relay:G5V-2
- added R10, R11, R21, R8, R9: 1M, rcl:0207/10
- added R12, R13, R14, R15: 50k, rcl:0207/10
- added R16, R17, R18, R19, R20: 70, rcl:0207/10
- added U$10, U$5: DA-2320, trafo:DIL06
- added U$11, U$12: VP0550L, transistor-fet:TO92L
- added U$4: UCC27425, texas:DIL08
- added U$6, U$7: VN0550L, transistor-fet:TO92L
- added X1: BU-SMA-V, con-coax:BU-SMA-V
Connections:
- new net +15V: C30.1, D9.C, K2.1, K2.8, K2.9, POWERGD1.1, U$4.6
- new net ENSW1: CONTROLGD2.1, D9.A, K2.16
- new net GND2: C30.2, C31.2, C32.2, CONTROLGD2.2, GND1.TP, GND13.TP, K2.11, K2.6, POWERGD1.2, U$10.6, U$4.3, U$5.6, X1.2, X1.3, X1.4, X1.5
- new net N$22: U$4.2, U$4.4, X1.1
- new net N$23: C25.1, U$4.7
- new net N$24: C26.1, U$4.5
- new net N$25: K2.4, U$4.1
- new net N$251: D21.A, R14.1, R18.2, U$6.2
- new net N$26: K2.13, U$4.8
- new net N$27: C24.1, U$5.2
- new net N$28: C27.1, U$5.3
- new net N$29: C28.1, U$10.2
- new net N$30: C29.1, U$10.3
- new net N$32: C28.2, D17.C, D21.C, R18.1
- new net N$33: C29.2, D18.C, D22.C, R19.1
- new net N$35: C27.2, D16.A, D20.A, R17.1
- new net N$36: C31.1, D10.C, D16.C, HV1.TP, R13.2, R8.2, U$11.3, U$5.4
- new net N$37: D13.A, D14.C, OUT1.TP, R10.2, R9.1, U$12.1, U$6.1
- new net N$38: U$10.5
- new net N$40: D17.A, R10.1, R11.2, R14.2, U$6.3, U$7.1
- new net N$41: D15.C, R12.2, R8.1, R9.2, U$11.1, U$12.3, U$5.5
- new net N$43: D19.C, R12.1, R16.2, U$12.2
- new net N$44: C24.2, D15.A, D19.A, R16.1
- new net N$45: D22.A, R15.1, R19.2, U$7.2
- new net N$46: D20.C, R13.1, R17.2, U$11.2
- new net N$47: R20.1, U$5.1
- new net N$48: R21.1, U$10.1
- new net N$49: C25.2, R20.2
- new net N$50: C26.2, R21.2
- new net N$51: C32.1, D12.A, D18.A, HV2.TP, R11.1, R15.2, U$10.4, U$7.3
- new net N$52: D10.A, D13.C
- new net N$53: D12.C, D14.A
Routing:
- net GND2: track 0.00 -> 98.9 mm, vias 0 -> 2
- net N$36: track 0.00 -> 98.4 mm
- net N$51: track 0.00 -> 95.6 mm
- net N$41: track 0.00 -> 87.6 mm
- net +15V: track 0.00 -> 77.6 mm
- net N$37: track 0.00 -> 56.6 mm
- net N$40: track 0.00 -> 55.3 mm
- net N$25: track 0.00 -> 38.6 mm
- net N$26: track 0.00 -> 38.1 mm
- net N$38: track 0.00 -> 28.8 mm
- net N$22: track 0.00 -> 26.2 mm
- net N$29: track 0.00 -> 21.5 mm
- net N$23: track 0.00 -> 20.6 mm
- net ENSW1: track 0.00 -> 18.9 mm
- net N$32: track 0.00 -> 16.5 mm
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- added copper zone on layer 16, net GND2
Other:
- board size 152.7 x 152.4 mm -> 255 x 152.4 mm
